Commit message: Added vulcano_torso_standalone

File: vulcano_torso_description/robots/vulcano_torso_standalone.urdf.xacro (robot description, xacro)
@@ -5,7 +5,12 @@
    <xacro:include filename="$(find vulcano_torso_description)/urdf/vulcano_torso.gazebo.xacro" />
    <xacro:include filename="$(find robotnik_sensors)/urdf/all_sensors.urdf.xacro" />
-   <xacro:torso prefix="vulcano_torso_">
+  <link name="world"/>
+  <joint name="fixed" type="fixed">
+    <parent link="world"/>
+    <child link="torso_base_link"/>
+  </joint>
+   <xacro:vulcano_torso prefix="torso_">
      <!-- origin xyz="0.427 0 0.152" rpy="0 0 0" /-->
      <origin xyz="0 0 0" rpy="0 0 0" />
-   </xacro:torso>
+   </xacro:vulcano_torso>
 </robot>

Commit message: Switched elevation and revolution joints prismatic and revolute type

File: vulcano_torso_description/robots/vulcano_torso_standalone.urdf.xacro (robot description, xacro)
@@ -14,5 +14,5 @@
         <parent link="world" />
         <child link="${prefix}base_link" />
-        <origin xyz="0.0 0.0 0.5" rpy="0.0 0.0 0.0" />
+        <origin xyz="0.0 0.0 0.6" rpy="0.0 0.0 0.0" />
     </joint>
     <xacro:vulcano_torso prefix="${prefix}" hq="${hq}">

File: vulcano_torso_description/urdf/common.gazebo.xacro (robot description, xacro)
@@ -5,5 +5,5 @@
     <gazebo>
       <plugin name="ros_control" filename="libgazebo_ros_control.so">
-        <robotNamespace>"${ns}"</robotNamespace>
+        <robotNamespace>${ns}</robotNamespace>
         <robotParam>robot_description</robotParam>
         <controlPeriod>0.001</controlPeriod>

File: vulcano_torso_description/urdf/torso/torso.urdf.xacro (robot description, xacro)
@@ -43,8 +43,8 @@
       </inertial>
     </link>
-    <joint name="${prefix}revolution_joint" type="fixed"> <!-- type="revolute" -->
+    <joint name="${prefix}revolution_joint" type="revolute">
       <!-- TODO: especificar zona muerta, limites de articulacion y parametros de simulacion -->
       <!--origin xyz="0 0 0" rpy="0 0 ${60*deg2rad}" /-->
-      <origin xyz="0 0 0" rpy="0 0 3.1415"/>
+      <origin xyz="0 0 0" rpy="0 0 ${PI}"/>
       <parent link="${prefix}guidance_base_link"/>
       <child link="${prefix}guidance_main_link"/>
@@ -53,4 +53,14 @@
       <dynamics friction="1000" damping="1000"/>
     </joint>
+	<transmission name="${prefix}revolution_trans">
+      <type>transmission_interface/SimpleTransmission</type>
+      <joint name="${prefix}revolution_joint">
+        <hardwareInterface>EffortJointInterface</hardwareInterface>
+      </joint>
+      <actuator name="${prefix}revolution_motor">
+        <mechanicalReduction>1</mechanicalReduction>
+        <hardwareInterface>EffortJointInterface</hardwareInterface>
+      </actuator>
+    </transmission>
     <link name="${prefix}guidance_main_link">
       <visual>
@@ -75,5 +85,5 @@
       </inertial>
     </link>
-    <joint name="${prefix}elevation_joint" type="fixed"> <!-- type="prismatic" -->
+    <joint name="${prefix}elevation_joint" type="prismatic">
       <!-- TODO: especificar limites de articulacion y parametros de simulacion -->
       <origin xyz="0 0 0.115" rpy="0 0 0"/>
@@ -83,4 +93,14 @@
       <limit lower="0" upper="0.739" effort="100" velocity="100"/>
     </joint>
+	<transmission name="${prefix}elevation_trans">
+      <type>transmission_interface/SimpleTransmission</type>
+      <joint name="${prefix}elevation_joint">
+        <hardwareInterface>EffortJointInterface</hardwareInterface>
+      </joint>
+      <actuator name="${prefix}elevation_motor">
+        <mechanicalReduction>1</mechanicalReduction>
+        <hardwareInterface>EffortJointInterface</hardwareInterface>
+      </actuator>
+    </transmission>
     <link name="${prefix}guidance_slide_link">
       <visual>
