Commit message: removed ns argument from urdfs

File: vulcano_description/robots/common.gazebo.xacro (robot description, xacro)
@@ -2,9 +2,9 @@
 <robot xmlns:xacro="http://ros.org/wiki/xacro">
   <!-- ros control plugin -->
-  <xacro:macro name="ros_control" params="ns">
+  <xacro:macro name="ros_control"> <!-- params="ns"> -->
     <gazebo>
       <plugin name="ros_control" filename="libgazebo_ros_control.so">
-        <robotNamespace>${ns}</robotNamespace>
-        <robotParam>robot_description</robotParam>
+        <!--<robotNamespace>${ns}</robotNamespace>-->
+        <!--<robotParam>robot_description</robotParam>-->
         <controlPeriod>0.001</controlPeriod>
 	    <robotSimType>gazebo_ros_control/DefaultRobotHWSim</robotSimType>

File: vulcano_torso_description/robots/vulcano_torso_standalone.urdf.xacro (robot description, xacro)
@@ -19,4 +19,4 @@
       <!-- origin xyz="0.427 0 0.152" rpy="0 0 0" /-->
     </xacro:vulcano_torso>
-    <xacro:ros_control ns="/vulcano_torso" />
+    <xacro:ros_control/> <!-- ns="/vulcano" / -->
 </robot>

File: vulcano_torso_description/urdf/common.gazebo.xacro (robot description, xacro)
@@ -2,9 +2,9 @@
 <robot xmlns:xacro="http://ros.org/wiki/xacro">
   <!-- ros control plugin -->
-  <xacro:macro name="ros_control" params="ns">
+  <xacro:macro name="ros_control"> <!-- params="ns" -->
     <gazebo>
       <plugin name="ros_control" filename="libgazebo_ros_control.so">
-        <robotNamespace>${ns}</robotNamespace>
-        <robotParam>robot_description</robotParam>
+        <!--<robotNamespace>${ns}</robotNamespace>-->
+        <!--<robotParam>robot_description</robotParam>-->
         <controlPeriod>0.001</controlPeriod>
 	    <robotSimType>gazebo_ros_control/DefaultRobotHWSim</robotSimType>
