Commit message: Modularization of vulcano_torso

File: vulcano_description/robots/vulcano_robot.urdf.xacro (robot description, xacro)
@@ -1,4 +1,4 @@
 <?xml version="1.0"?>
-<robot xmlns:xacro="http://www.ros.org/wiki/xacro" name="vulcano">
+<robot name="vulcano" xmlns:xacro="http://www.ros.org/wiki/xacro">
   <xacro:property name="PI" value="3.1415926535897931"/>
   <!-- ***************** -->
@@ -24,5 +24,4 @@
     <origin xyz="-0.1637 0.275533 0.021967" rpy="0 ${-PI/4.0} ${-PI/2.0}"/>  <!-- TODO: set correct orientation -->
     <parent link="torso_tkd668_link"/>
-    <!--child link="right_arm_rotate_base_link"/-->
     <child link="right_arm_base_link"/>
   </joint>

File: vulcano_torso_description/robots/vulcano_torso_standalone.urdf.xacro (robot description, xacro)
@@ -1,16 +1,22 @@
 <?xml version="1.0"?>
-<robot name="vulcano" xmlns:xacro="http://ros.org/wiki/xacro"> <!-- TODO: check robot name -->
-   <!-- Include all component files -->
-   <xacro:include filename="$(find vulcano_torso_description)/urdf/vulcano_torso.urdf.xacro" />
-   <xacro:include filename="$(find vulcano_torso_description)/urdf/vulcano_torso.gazebo.xacro" />
-   <xacro:include filename="$(find robotnik_sensors)/urdf/all_sensors.urdf.xacro" />
-  <link name="world"/>
-  <joint name="fixed" type="fixed">
-    <parent link="world"/>
-    <child link="torso_base_link"/>
-  </joint>
-   <xacro:vulcano_torso prefix="torso_">
-     <!-- origin xyz="0.427 0 0.152" rpy="0 0 0" /-->
-     <origin xyz="0 0 0" rpy="0 0 0" />
-   </xacro:vulcano_torso>
+<robot name="vulcano_torso" xmlns:xacro="http://ros.org/wiki/xacro"> <!-- TODO: check robot name -->
+	<!-- ***************** -->
+	<!-- Imported elements -->
+	<!-- ***************** -->
+	<!-- First we import all posible elements defined in the urdf.xacro files. All these elements are defined as macro:xacros -->
+	<!-- Import vulcano torso elements -->
+    <xacro:include filename="$(find vulcano_torso_description)/urdf/vulcano_torso.urdf.xacro" />
+    <xacro:include filename="$(find vulcano_torso_description)/urdf/common.gazebo.xacro" />
+    <xacro:property name="prefix" value="" />
+    <xacro:property name="hq" value="true" />
+    <link name="world" />
+    <joint name="world_joint" type="fixed">
+        <parent link="world" />
+        <child link="${prefix}base_link" />
+        <origin xyz="0.0 0.0 0.5" rpy="0.0 0.0 0.0" />
+    </joint>
+    <xacro:vulcano_torso prefix="${prefix}" hq="${hq}">
+      <!-- origin xyz="0.427 0 0.152" rpy="0 0 0" /-->
+    </xacro:vulcano_torso>
+    <xacro:ros_control ns="/vulcano_torso" />
 </robot>

File: vulcano_torso_description/urdf/vulcano_torso.urdf.xacro (robot description, xacro)
@@ -1,131 +1,13 @@
 <?xml version="1.0"?>
-<robot name="vulcano_torso" xmlns:xacro="http://ros.org/wiki/xacro">
-  <xacro:property name="PI" value="3.1415926535897931"/>
-  <xacro:property name="deg2rad" value="0.01745329251"/>
-  <xacro:property name="elevation_max_longitude" value="0.7"/>
-  <xacro:property name="z_elevation_joint" value="0.442"/>
-  <!-- Define the torso -->
-  <xacro:macro name="vulcano_torso" params="prefix *origin">
-    <link name="${prefix}base_link">
-      <inertial>
-        <origin xyz="0 0 0" rpy="0 0 0 "/>
-        <mass value="5"/> <!-- TODO: check masses -->
-        <inertia ixx="1.0" ixy="0.0" ixz="0.0" iyy="1.0" iyz="0.0" izz="1.0"/>
-      </inertial>
-    </link>
-    <joint name="${prefix}guidance_base_joint" type="fixed">
-      <!--<origin xyz="0.47 0 0.474" rpy="0 0 0"/>-->
-      <origin xyz="0.0 0.0 0.0" rpy="0 0 0"/>
-      <parent link="${prefix}base_link"/>
-      <child link="${prefix}guidance_base_link"/>
-      <axis xyz="0 0 1"/>
-    </joint>
-    <link name="${prefix}guidance_base_link">
-      <visual>
-        <origin xyz="0 0 0" rpy="0 0 0"/>
-        <geometry>
-          <mesh filename="package://vulcano_torso_description/meshes/guidance_base.stl"/>
-        </geometry>
-       <material name="darkgrey">
-         <color rgba="0.1 0.1 0.1 1"/>
-       </material>
-      </visual>
-      <collision>
-        <origin xyz="0 0 0" rpy="0 0 0"/>
-        <geometry>
-          <mesh filename="package://vulcano_torso_description/meshes/guidance_base.stl"/>
-        </geometry>
-      </collision>
-      <inertial>
-        <origin xyz="0 0 0" rpy="0 0 0"/>
-        <mass value="5"/>
-        <inertia ixx="1.0" ixy="0.0" ixz="0.0" iyy="1.0" iyz="0.0" izz="1.0"/>
-      </inertial>
-    </link>
-    <joint name="${prefix}revolution_joint" type="revolute">
-      <!-- TODO: especificar zona muerta, limites de articulacion y parametros de simulacion -->
-      <!--origin xyz="0 0 0" rpy="0 0 ${60*deg2rad}" /-->
-      <origin xyz="0 0 0" rpy="0 0 3.1415"/>
-      <parent link="${prefix}guidance_base_link"/>
-      <child link="${prefix}guidance_main_link"/>
-      <axis xyz="0 0 1"/>
-      <limit lower="${-172*deg2rad}" upper="${172*deg2rad}" effort="100" velocity="100"/>
-      <dynamics friction="1000" damping="1000"/>
-    </joint>
-    <link name="${prefix}guidance_main_link">
-      <visual>
-        <origin xyz="0 0 0" rpy="0 0 0"/>
-        <geometry>
-          <mesh filename="package://vulcano_torso_description/meshes/guidance_main.stl"/>
-        </geometry>
-       <material name="darkgrey">
-         <color rgba="0.1 0.1 0.1 1"/>
-       </material>
-      </visual>
-      <collision>
-        <origin xyz="0 0 0" rpy="0 0 0"/>
-        <geometry>
-          <mesh filename="package://vulcano_torso_description/meshes/guidance_main.stl"/>
-        </geometry>
-      </collision>
-      <inertial>
-        <origin xyz="0 0 0" rpy="0 0 0"/>
-        <mass value="5"/>
-        <inertia ixx="1.0" ixy="0.0" ixz="0.0" iyy="1.0" iyz="0.0" izz="1.0"/>
-      </inertial>
-    </link>
-    <joint name="${prefix}elevation_joint" type="prismatic">
-      <!-- TODO: especificar limites de articulacion y parametros de simulacion -->
-      <origin xyz="0 0 0.115" rpy="0 0 0"/>
-      <parent link="${prefix}guidance_main_link"/>
-      <child link="${prefix}guidance_slide_link"/>
-      <axis xyz="0 0 1"/>
-      <limit lower="0" upper="0.739" effort="100" velocity="100"/>
-    </joint>
-    <link name="${prefix}guidance_slide_link">
-      <visual>
-        <origin xyz="0 0 0" rpy="0 0 0"/>
-        <geometry>
-          <mesh filename="package://vulcano_torso_description/meshes/guidance_slide.stl"/>
-        </geometry>
-       <material name="darkgrey">
-         <color rgba="0.1 0.1 0.1 1"/>
-       </material>
-      </visual>
-      <collision>
-        <origin xyz="0 0 0" rpy="0 0 0"/>
-        <geometry>
-          <mesh filename="package://vulcano_torso_description/meshes/guidance_slide.stl"/>
-        </geometry>
-      </collision>
-      <inertial>
-        <origin xyz="0 0 0" rpy="0 0 0"/>
-        <mass value="1"/>
-        <inertia ixx="1.0" ixy="0.0" ixz="0.0" iyy="1.0" iyz="0.0" izz="1.0"/>
-      </inertial>
-    </link>
-    <joint name="${prefix}tkd668_joint" type="fixed">
-      <origin xyz="0.164 0 0.449" rpy="0 0 0"/>
-      <parent link="${prefix}guidance_slide_link"/>
-      <child link="${prefix}tkd668_link"/>
-      <axis xyz="0 0 1"/>
-    </joint>
-    <link name="${prefix}tkd668_link">
-      <visual>
-        <origin xyz="0 0 0" rpy="0 0 0"/>
-        <geometry>
-          <mesh filename="package://vulcano_torso_description/meshes/tkd668.stl"/>
-        </geometry>
-       <material name="darkgrey">
-         <color rgba="0.1 0.1 0.1 1"/>
-       </material>
-      </visual>
-      <collision>
-        <origin xyz="0 0 0" rpy="0 0 0"/>
-        <geometry>
-          <mesh filename="package://vulcano_torso_description/meshes/tkd668.stl"/>
-        </geometry>
-      </collision>
-    </link>
-  </xacro:macro>
+<robot xmlns:xacro="http://ros.org/wiki/xacro">
+    <!-- ***************** -->
+    <!-- Imported elements -->
+    <!-- ***************** -->
+    <!-- First we import all posible elements defined in the urdf.xacro files. All these elements are defined as macro:xacros -->
+    <!-- Include vulcano torso elements -->
+    <xacro:include filename="$(find vulcano_torso_description)/urdf/torso/torso.urdf.xacro"/>
+    <xacro:include filename="$(find robotnik_sensors)/urdf/all_sensors.urdf.xacro" />
+    <xacro:macro name="vulcano_torso" params="prefix hq">
+        <xacro:torso prefix="${prefix}" hq="${hq}"/>
+    </xacro:macro>
 </robot>

Commit message: Updated vulcano_description and vulcano_torso_description

File: vulcano_description/robots/vulcano_robot.urdf.xacro (robot description, xacro)
@@ -7,10 +7,15 @@
   <!-- First we import all posible elements defined in the urdf.xacro files. All these elements are defined as macro:xacros -->
   <!-- Import vulcano base -->
-  <xacro:include filename="$(find vulcano_base_description)/robots/vulcano_base.urdf.xacro" />
+  <xacro:include filename="$(find vulcano_base_description)/urdf/vulcano_base.urdf.xacro" />
   <!-- Import vulcano torso -->
-  <xacro:include filename="$(find vulcano_torso_description)/robots/vulcano_torso.urdf.xacro"/>
+  <xacro:include filename="$(find vulcano_torso_description)/urdf/vulcano_torso.urdf.xacro"/>
   <!-- Import UR10 -->
   <xacro:include filename="$(find ur_description)/urdf/ur10.urdf.xacro"/>
-  <xacro:include filename="$(find ur_description)/urdf/common.gazebo.xacro"/>
+  <!--<xacro:include filename="$(find ur_description)/urdf/common.gazebo.xacro"/>-->
+  <!-- Import common gazebo elements -->
+  <xacro:include filename="$(find vulcano_description)/robots/common.gazebo.xacro" />
+  <xacro:property name="hq" value="true" />
+  <xacro:property name="publish_bf" value="true" />
+  <xacro:vulcano_base prefix="" publish_bf="${publish_bf}" hq="${hq}"/>
   <!-- Fix torso to base -->
   <joint name="base_torso_joint" type="fixed">
@@ -20,4 +25,5 @@
     <axis xyz="0 0 0"/>
   </joint>
+  <xacro:vulcano_torso prefix="" hq="${hq}" />
   <!-- Fix right arm to torso -->
   <joint name="torso_right_arm_base_joint" type="fixed">
@@ -34,3 +40,4 @@
   </joint>
   <xacro:ur10_robot prefix="left_arm_" joint_limited="true"/>
+  <xacro:ros_control ns="/vulcano"/>
 </robot>

File: vulcano_torso_description/robots/vulcano_torso_standalone.urdf.xacro (robot description, xacro)
@@ -13,5 +13,5 @@
     <joint name="world_joint" type="fixed">
         <parent link="world" />
-        <child link="${prefix}base_link" />
+        <child link="${prefix}torso_base_link" />
         <origin xyz="0.0 0.0 0.6" rpy="0.0 0.0 0.0" />
     </joint>

File: vulcano_torso_description/urdf/torso/torso.urdf.xacro (robot description, xacro)
@@ -7,5 +7,5 @@
   <!-- Define the torso -->
   <xacro:macro name="torso" params="prefix hq">
-    <link name="${prefix}base_link">
+    <link name="${prefix}torso_base_link">
       <inertial>
         <origin xyz="0 0 0" rpy="0 0 0 "/>
@@ -14,12 +14,12 @@
       </inertial>
     </link>
-    <joint name="${prefix}guidance_base_joint" type="fixed">
+    <joint name="${prefix}torso_guidance_base_joint" type="fixed">
       <!--<origin xyz="0.47 0 0.474" rpy="0 0 0"/>-->
       <origin xyz="0.0 0.0 0.0" rpy="0 0 0"/>
-      <parent link="${prefix}base_link"/>
-      <child link="${prefix}guidance_base_link"/>
+      <parent link="${prefix}torso_base_link"/>
+      <child link="${prefix}torso_guidance_base_link"/>
       <axis xyz="0 0 1"/>
     </joint>
-    <link name="${prefix}guidance_base_link">
+    <link name="${prefix}torso_guidance_base_link">
       <visual>
         <origin xyz="0 0 0" rpy="0 0 0"/>
@@ -43,25 +43,26 @@
       </inertial>
     </link>
-    <joint name="${prefix}revolution_joint" type="revolute">
+    <joint name="${prefix}torso_revolution_joint" type="revolute">
       <!-- TODO: especificar zona muerta, limites de articulacion y parametros de simulacion -->
       <!--origin xyz="0 0 0" rpy="0 0 ${60*deg2rad}" /-->
       <origin xyz="0 0 0" rpy="0 0 ${PI}"/>
-      <parent link="${prefix}guidance_base_link"/>
-      <child link="${prefix}guidance_main_link"/>
+      <parent link="${prefix}torso_guidance_base_link"/>
+      <child link="${prefix}torso_guidance_main_link"/>
       <axis xyz="0 0 1"/>
       <limit lower="${-172*deg2rad}" upper="${172*deg2rad}" effort="100" velocity="100"/>
       <dynamics friction="1000" damping="1000"/>
     </joint>
-	<transmission name="${prefix}revolution_trans">
+	<transmission name="${prefix}torso_revolution_trans">
       <type>transmission_interface/SimpleTransmission</type>
-      <joint name="${prefix}revolution_joint">
-        <hardwareInterface>EffortJointInterface</hardwareInterface>
+      <joint name="${prefix}torso_revolution_joint">
+        <!--<hardwareInterface>EffortJointInterface</hardwareInterface>-->
+        <hardwareInterface>PositionJointInterface</hardwareInterface><!-- TODO: PositionJointInterface? EffortJointInterface? -->
       </joint>
-      <actuator name="${prefix}revolution_motor">
+      <actuator name="${prefix}torso_revolution_motor">
         <mechanicalReduction>1</mechanicalReduction>
         <hardwareInterface>EffortJointInterface</hardwareInterface>
       </actuator>
     </transmission>
-    <link name="${prefix}guidance_main_link">
+    <link name="${prefix}torso_guidance_main_link">
       <visual>
         <origin xyz="0 0 0" rpy="0 0 0"/>
@@ -85,23 +86,24 @@
       </inertial>
     </link>
-    <joint name="${prefix}elevation_joint" type="prismatic">
+    <joint name="${prefix}torso_elevation_joint" type="prismatic">
       <!-- TODO: especificar limites de articulacion y parametros de simulacion -->
       <origin xyz="0 0 0.115" rpy="0 0 0"/>
-      <parent link="${prefix}guidance_main_link"/>
-      <child link="${prefix}guidance_slide_link"/>
+      <parent link="${prefix}torso_guidance_main_link"/>
+      <child link="${prefix}torso_guidance_slide_link"/>
       <axis xyz="0 0 1"/>
       <limit lower="0" upper="0.739" effort="100" velocity="100"/>
     </joint>
-	<transmission name="${prefix}elevation_trans">
+	<transmission name="${prefix}torso_elevation_trans">
       <type>transmission_interface/SimpleTransmission</type>
-      <joint name="${prefix}elevation_joint">
-        <hardwareInterface>EffortJointInterface</hardwareInterface>
+      <joint name="${prefix}torso_elevation_joint">
+        <!--<hardwareInterface>EffortJointInterface</hardwareInterface>-->
+        <hardwareInterface>PositionJointInterface</hardwareInterface><!-- TODO: PositionJointInterface? EffortJointInterface? -->
       </joint>
-      <actuator name="${prefix}elevation_motor">
+      <actuator name="${prefix}torso_elevation_motor">
         <mechanicalReduction>1</mechanicalReduction>
         <hardwareInterface>EffortJointInterface</hardwareInterface>
       </actuator>
     </transmission>
-    <link name="${prefix}guidance_slide_link">
+    <link name="${prefix}torso_guidance_slide_link">
       <visual>
         <origin xyz="0 0 0" rpy="0 0 0"/>
@@ -125,11 +127,11 @@
       </inertial>
     </link>
-    <joint name="${prefix}tkd668_joint" type="fixed">
+    <joint name="${prefix}torso_tkd668_joint" type="fixed">
       <origin xyz="0.164 0 0.449" rpy="0 0 0"/>
-      <parent link="${prefix}guidance_slide_link"/>
-      <child link="${prefix}tkd668_link"/>
+      <parent link="${prefix}torso_guidance_slide_link"/>
+      <child link="${prefix}torso_tkd668_link"/>
       <axis xyz="0 0 1"/>
     </joint>
-    <link name="${prefix}tkd668_link">
+    <link name="${prefix}torso_tkd668_link">
       <visual>
         <origin xyz="0 0 0" rpy="0 0 0"/>

Commit message: vulcano_torso_description: corrected bug and added tube support of arms

File: vulcano_description/robots/vulcano_robot.urdf.xacro (robot description, xacro)
@@ -35,9 +35,17 @@
   <!-- Fix left arm to torso -->
   <joint name="torso_left_arm_base_joint" type="fixed">
-    <origin xyz="-0.1637 -0.275533 0.021967" rpy="0 ${PI/4.0} ${-PI/2.0}"/>
+    <origin xyz="-0.1622 -0.275533 0.021967" rpy="0 ${PI/4.0} ${-PI/2.0}"/>
     <parent link="torso_tkd668_link"/>
     <child link="left_arm_base_link"/>
   </joint>
   <xacro:ur10_robot prefix="left_arm_" joint_limited="true"/>
+  <xacro:tube_support prefix="left_arm_ee_" parent="left_arm_ee_link">
+    <origin xyz="0.014 0 0.0975" rpy="0 0 0"/>
+    <box size="0.102 0.075 0.075" />
+  </xacro:tube_support>
+  <xacro:tube_support prefix="right_arm_ee_" parent="right_arm_ee_link">
+    <origin xyz="0.014 0 0.0975" rpy="0 0 0"/>
+    <box size="0.102 0.075 0.075" />
+  </xacro:tube_support>
   <xacro:ros_control />
 </robot>

File: vulcano_torso_description/urdf/guidance/guidance.urdf.xacro (robot description, xacro)
@@ -36,10 +36,9 @@
     </link>
     <joint name="${prefix}torso_guidance_revolution_joint" type="revolute">
-      <!-- TODO: especificar zona muerta, limites de articulacion y parametros de simulacion -->
       <origin xyz="0 0 0" rpy="0 0 ${PI}"/>
       <parent link="${prefix}torso_guidance_base_link"/>
       <child link="${prefix}torso_guidance_revolution_link"/>
       <axis xyz="0 0 1"/>
-      <limit lower="${-135*deg2rad}" upper="${225*deg2rad}" effort="100" velocity="100"/>
+      <limit lower="${-180*deg2rad}" upper="${180*deg2rad}" effort="100" velocity="100"/>
       <dynamics friction="1000" damping="1000"/>
     </joint>
@@ -47,10 +46,8 @@
       <type>transmission_interface/SimpleTransmission</type>
       <joint name="${prefix}torso_guidance_revolution_joint">
-        <!--<hardwareInterface>EffortJointInterface</hardwareInterface>-->
-        <hardwareInterface>PositionJointInterface</hardwareInterface> <!-- TODO: PositionJointInterface? EffortJointInterface?  VelocityJointInterface? -->
+        <hardwareInterface>PositionJointInterface</hardwareInterface>
       </joint>
       <actuator name="${prefix}torso_guidance_revolution_motor">
         <mechanicalReduction>1</mechanicalReduction>
-        <hardwareInterface>EffortJointInterface</hardwareInterface>
       </actuator>
     </transmission>
@@ -88,10 +85,8 @@
       <type>transmission_interface/SimpleTransmission</type>
       <joint name="${prefix}torso_guidance_elevation_joint">
-        <!--<hardwareInterface>EffortJointInterface</hardwareInterface>-->
-        <hardwareInterface>PositionJointInterface</hardwareInterface> <!-- TODO: PositionJointInterface? EffortJointInterface?  VelocityJointInterface? -->
+        <hardwareInterface>PositionJointInterface</hardwareInterface>
       </joint>
       <actuator name="${prefix}torso_guidance_elevation_motor">
         <mechanicalReduction>1</mechanicalReduction>
-        <hardwareInterface>EffortJointInterface</hardwareInterface>
       </actuator>
     </transmission>

File: vulcano_torso_description/urdf/vulcano_torso.urdf.xacro (robot description, xacro)
@@ -9,4 +9,5 @@
     <xacro:include filename="$(find vulcano_torso_description)/urdf/guidance/guidance.urdf.xacro"/>
     <xacro:include filename="$(find vulcano_torso_description)/urdf/pantilt/pantilt.urdf.xacro"/>
+    <xacro:include filename="$(find vulcano_torso_description)/urdf/tube_support/tube_support.urdf.xacro"/>
     <xacro:include filename="$(find robotnik_sensors)/urdf/all_sensors.urdf.xacro" />
     <xacro:macro name="vulcano_torso" params="prefix hq"> <!-- TODO: check hq variable -->

Commit message: descriptions: corrected models

File: vulcano_description/robots/vulcano_robot.urdf.xacro (robot description, xacro)
@@ -28,5 +28,5 @@
   <!-- Fix right arm to torso -->
   <joint name="torso_right_arm_base_joint" type="fixed">
-    <origin xyz="-0.1637 0.275533 0.021967" rpy="0 ${-PI/4.0} ${-PI/2.0}"/>  <!-- TODO: set correct orientation -->
+    <origin xyz="-0.1622 0.275533 0.021967" rpy="0 ${-PI/4.0} ${-PI/2.0}"/>  <!-- TODO: set correct orientation -->
     <parent link="torso_tkd668_link"/>
     <child link="right_arm_base_link"/>
@@ -41,10 +41,10 @@
   <xacro:ur10_robot prefix="left_arm_" joint_limited="true"/>
   <xacro:tube_support prefix="left_arm_ee_" parent="left_arm_ee_link">
-    <origin xyz="0.014 0 0.0975" rpy="0 0 0"/>
-    <box size="0.102 0.075 0.075" />
+    <origin xyz="0.012 0 0.0975" rpy="0 0 0"/>
+    <box size="0.075 0.075 0.075" />
   </xacro:tube_support>
   <xacro:tube_support prefix="right_arm_ee_" parent="right_arm_ee_link">
-    <origin xyz="0.014 0 0.0975" rpy="0 0 0"/>
-    <box size="0.102 0.075 0.075" />
+    <origin xyz="0.012 0 0.0975" rpy="0 0 0"/>
+    <box size="0.075 0.075 0.075" />
   </xacro:tube_support>
   <xacro:ros_control />

File: vulcano_torso_description/urdf/guidance/guidance.urdf.xacro (robot description, xacro)
@@ -40,5 +40,5 @@
       <child link="${prefix}torso_guidance_revolution_link"/>
       <axis xyz="0 0 1"/>
-      <limit lower="${-180*deg2rad}" upper="${180*deg2rad}" effort="100" velocity="100"/>
+      <limit lower="${-180*deg2rad}" upper="${180*deg2rad}" effort="100" velocity="0.4"/>
       <dynamics friction="1000" damping="1000"/>
     </joint>
@@ -79,5 +79,5 @@
       <child link="${prefix}torso_guidance_elevation_link"/>
       <axis xyz="0 0 1"/>
-      <limit lower="0.0" upper="0.68" effort="100" velocity="100"/>
+      <limit lower="0.0" upper="0.68" effort="100" velocity="0.08"/>
       <dynamics friction="100000" damping="10000"/>
     </joint>

Commit message: description: ported from indigo-devel

File: vulcano_description/robots/vulcano_robot.urdf.xacro (robot description, xacro)
@@ -20,5 +20,5 @@
   <!-- Fix torso to base -->
   <joint name="base_torso_joint" type="fixed">
-    <origin xyz="0.5607 0.0 0.4845" rpy="0.0 0.0 0.0"/>
+    <origin xyz="0.47 0.0 0.474" rpy="0.0 0.0 0.0"/>
     <parent link="base_link"/>
     <child link="torso_base_link"/>
@@ -28,6 +28,6 @@
   <!-- Fix right arm to torso -->
   <joint name="torso_right_arm_base_joint" type="fixed">
-    <origin xyz="0.16870 0.28753 -0.12303" rpy="0 ${-PI/4.0} ${-PI/2.0}"/>
-    <parent link="torso_guidance_elevation_link"/>
+    <origin xyz="-0.1622 0.275533 0.021967" rpy="0 ${-PI/4.0} ${-PI/2.0}"/>  <!-- TODO: set correct orientation -->
+    <parent link="torso_tkd668_link"/>
     <child link="right_arm_base_link"/>
   </joint>
@@ -35,6 +35,6 @@
   <!-- Fix left arm to torso -->
   <joint name="torso_left_arm_base_joint" type="fixed">
-    <origin xyz="0.16870 -0.28753 -0.12303" rpy="0 ${PI/4.0} ${-PI/2.0}"/>
-    <parent link="torso_guidance_elevation_link"/>
+    <origin xyz="-0.1622 -0.275533 0.021967" rpy="0 ${PI/4.0} ${-PI/2.0}"/>
+    <parent link="torso_tkd668_link"/>
     <child link="left_arm_base_link"/>
   </joint>
