Commit message: Modified left/right arm xacro to avoid overwritting offsets

File: vulcano_calibrated_ur_description/urdf/calibrated_ur10_vulcano_right_arm.urdf.xacro (robot description, xacro)
@@ -55,46 +55,46 @@
     </xacro:macro>
     <!-- calibrations offsets -->
-    <xacro:property name="shoulder_pan_joint_offset" value="-4.00915e-05" />
-    <xacro:property name="shoulder_lift_joint_offset" value="1.46569e-05" />
-    <xacro:property name="elbow_joint_offset" value="-0.000115152" />
-    <xacro:property name="wrist_1_joint_offset" value="5.33759e-05" />
-    <xacro:property name="wrist_2_joint_offset" value="0.000187537" />
-    <xacro:property name="wrist_3_joint_offset" value="0.000183181" />
-    <xacro:property name="shoulder_pan_joint_x_offset" value="-8.47099e-08" />
-    <xacro:property name="shoulder_pan_joint_y_offset" value="-7.51021e-07" />
-    <xacro:property name="shoulder_pan_joint_z_offset" value="0.000228625" />
-    <xacro:property name="shoulder_pan_joint_a_offset" value="-8.00303e-07" />
-    <xacro:property name="shoulder_pan_joint_b_offset" value="2.68717e-07" />
-    <xacro:property name="shoulder_pan_joint_c_offset" value="-5.77789e-06" />
-    <xacro:property name="shoulder_lift_joint_x_offset" value="4.43342e-05" />
-    <xacro:property name="shoulder_lift_joint_y_offset" value="-0.000118657" />
-    <xacro:property name="shoulder_lift_joint_z_offset" value="0.000228626" />
-    <xacro:property name="shoulder_lift_joint_a_offset" value="-0.000531359" />
-    <xacro:property name="shoulder_lift_joint_b_offset" value="1.30762e-05" />
-    <xacro:property name="shoulder_lift_joint_c_offset" value="-9.64047e-06" />
-    <xacro:property name="elbow_joint_x_offset" value="0.000117534" />
-    <xacro:property name="elbow_joint_y_offset" value="-0.00011866" />
-    <xacro:property name="elbow_joint_z_offset" value="0.000422057" />
-    <xacro:property name="elbow_joint_a_offset" value="0.000625564" />
-    <xacro:property name="elbow_joint_b_offset" value="8.31801e-06" />
-    <xacro:property name="elbow_joint_c_offset" value="-0.000723379" />
-    <xacro:property name="wrist_1_joint_x_offset" value="-0.000117352" />
-    <xacro:property name="wrist_1_joint_y_offset" value="-0.000118652" />
-    <xacro:property name="wrist_1_joint_z_offset" value="-0.000893361" />
-    <xacro:property name="wrist_1_joint_a_offset" value="0.00103716" />
-    <xacro:property name="wrist_1_joint_b_offset" value="-0.000115892" />
-    <xacro:property name="wrist_1_joint_c_offset" value="0.0043396" />
-    <xacro:property name="wrist_2_joint_x_offset" value="0.000115388" />
-    <xacro:property name="wrist_2_joint_y_offset" value="-0.000118642" />
-    <xacro:property name="wrist_2_joint_z_offset" value="1.7781e-05" />
-    <xacro:property name="wrist_2_joint_a_offset" value="-0.000411286" />
-    <xacro:property name="wrist_2_joint_b_offset" value="0.000153786" />
-    <xacro:property name="wrist_2_joint_c_offset" value="-0.000410757" />
-    <xacro:property name="wrist_3_joint_x_offset" value="-3.99584e-05" />
-    <xacro:property name="wrist_3_joint_y_offset" value="-0.000288006" />
-    <xacro:property name="wrist_3_joint_z_offset" value="1.78033e-05" />
-    <xacro:property name="wrist_3_joint_a_offset" value="0.000104033" />
-    <xacro:property name="wrist_3_joint_b_offset" value="-0.000202165" />
-    <xacro:property name="wrist_3_joint_c_offset" value="0.000150637" />
+    <xacro:property name="right_arm_shoulder_pan_joint_offset" value="-4.00915e-05" />
+    <xacro:property name="right_arm_shoulder_lift_joint_offset" value="1.46569e-05" />
+    <xacro:property name="right_arm_elbow_joint_offset" value="-0.000115152" />
+    <xacro:property name="right_arm_wrist_1_joint_offset" value="5.33759e-05" />
+    <xacro:property name="right_arm_wrist_2_joint_offset" value="0.000187537" />
+    <xacro:property name="right_arm_wrist_3_joint_offset" value="0.000183181" />
+    <xacro:property name="right_arm_shoulder_pan_joint_x_offset" value="-8.47099e-08" />
+    <xacro:property name="right_arm_shoulder_pan_joint_y_offset" value="-7.51021e-07" />
+    <xacro:property name="right_arm_shoulder_pan_joint_z_offset" value="0.000228625" />
+    <xacro:property name="right_arm_shoulder_pan_joint_a_offset" value="-8.00303e-07" />
+    <xacro:property name="right_arm_shoulder_pan_joint_b_offset" value="2.68717e-07" />
+    <xacro:property name="right_arm_shoulder_pan_joint_c_offset" value="-5.77789e-06" />
+    <xacro:property name="right_arm_shoulder_lift_joint_x_offset" value="4.43342e-05" />
+    <xacro:property name="right_arm_shoulder_lift_joint_y_offset" value="-0.000118657" />
+    <xacro:property name="right_arm_shoulder_lift_joint_z_offset" value="0.000228626" />
+    <xacro:property name="right_arm_shoulder_lift_joint_a_offset" value="-0.000531359" />
+    <xacro:property name="right_arm_shoulder_lift_joint_b_offset" value="1.30762e-05" />
+    <xacro:property name="right_arm_shoulder_lift_joint_c_offset" value="-9.64047e-06" />
+    <xacro:property name="right_arm_elbow_joint_x_offset" value="0.000117534" />
+    <xacro:property name="right_arm_elbow_joint_y_offset" value="-0.00011866" />
+    <xacro:property name="right_arm_elbow_joint_z_offset" value="0.000422057" />
+    <xacro:property name="right_arm_elbow_joint_a_offset" value="0.000625564" />
+    <xacro:property name="right_arm_elbow_joint_b_offset" value="8.31801e-06" />
+    <xacro:property name="right_arm_elbow_joint_c_offset" value="-0.000723379" />
+    <xacro:property name="right_arm_wrist_1_joint_x_offset" value="-0.000117352" />
+    <xacro:property name="right_arm_wrist_1_joint_y_offset" value="-0.000118652" />
+    <xacro:property name="right_arm_wrist_1_joint_z_offset" value="-0.000893361" />
+    <xacro:property name="right_arm_wrist_1_joint_a_offset" value="0.00103716" />
+    <xacro:property name="right_arm_wrist_1_joint_b_offset" value="-0.000115892" />
+    <xacro:property name="right_arm_wrist_1_joint_c_offset" value="0.0043396" />
+    <xacro:property name="right_arm_wrist_2_joint_x_offset" value="0.000115388" />
+    <xacro:property name="right_arm_wrist_2_joint_y_offset" value="-0.000118642" />
+    <xacro:property name="right_arm_wrist_2_joint_z_offset" value="1.7781e-05" />
+    <xacro:property name="right_arm_wrist_2_joint_a_offset" value="-0.000411286" />
+    <xacro:property name="right_arm_wrist_2_joint_b_offset" value="0.000153786" />
+    <xacro:property name="right_arm_wrist_2_joint_c_offset" value="-0.000410757" />
+    <xacro:property name="right_arm_wrist_3_joint_x_offset" value="-3.99584e-05" />
+    <xacro:property name="right_arm_wrist_3_joint_y_offset" value="-0.000288006" />
+    <xacro:property name="right_arm_wrist_3_joint_z_offset" value="1.78033e-05" />
+    <xacro:property name="right_arm_wrist_3_joint_a_offset" value="0.000104033" />
+    <xacro:property name="right_arm_wrist_3_joint_b_offset" value="-0.000202165" />
+    <xacro:property name="right_arm_wrist_3_joint_c_offset" value="0.000150637" />
     <xacro:macro name="right_arm_ur10_robot" params="prefix joint_limited shoulder_pan_lower_limit:=${-pi} shoulder_pan_upper_limit:=${pi} shoulder_lift_lower_limit:=${-pi} shoulder_lift_upper_limit:=${pi} elbow_joint_lower_limit:=${-pi} elbow_joint_upper_limit:=${pi} wrist_1_lower_limit:=${-pi} wrist_1_upper_limit:=${pi} wrist_2_lower_limit:=${-pi} wrist_2_upper_limit:=${pi} wrist_3_lower_limit:=${-pi} wrist_3_upper_limit:=${pi}">
         <link name="${prefix}base_link">
@@ -117,5 +117,5 @@
         </link>
         <joint name="${prefix}shoulder_pan_offset_joint" type="fixed">
-            <origin xyz="${shoulder_pan_joint_x_offset} ${shoulder_pan_joint_y_offset} ${shoulder_pan_joint_z_offset}" rpy="${shoulder_pan_joint_a_offset} ${shoulder_pan_joint_b_offset} ${shoulder_pan_joint_c_offset}" />
+            <origin xyz="${right_arm_shoulder_pan_joint_x_offset} ${right_arm_shoulder_pan_joint_y_offset} ${right_arm_shoulder_pan_joint_z_offset}" rpy="${right_arm_shoulder_pan_joint_a_offset} ${right_arm_shoulder_pan_joint_b_offset} ${right_arm_shoulder_pan_joint_c_offset}" />
             <parent link="${prefix}base_link" />
             <child link="${prefix}shoulder_pan_offset_link" />
@@ -125,5 +125,5 @@
             <parent link="${prefix}shoulder_pan_offset_link" />
             <child link="${prefix}shoulder_link" />
-            <origin xyz="0.0 0.0 ${shoulder_height}" rpy="0.0 0.0 ${shoulder_pan_joint_offset}" />
+            <origin xyz="0.0 0.0 ${shoulder_height}" rpy="0.0 0.0 ${right_arm_shoulder_pan_joint_offset}" />
             <axis xyz="0 0 1" />
             <calibration rising="0.0" />
@@ -155,5 +155,5 @@
         </link>
         <joint name="${prefix}shoulder_lift_offset_joint" type="fixed">
-            <origin xyz="${shoulder_lift_joint_x_offset} ${shoulder_lift_joint_y_offset} ${shoulder_lift_joint_z_offset}" rpy="${shoulder_lift_joint_a_offset} ${shoulder_lift_joint_b_offset} ${shoulder_lift_joint_c_offset}" />
+            <origin xyz="${right_arm_shoulder_lift_joint_x_offset} ${right_arm_shoulder_lift_joint_y_offset} ${right_arm_shoulder_lift_joint_z_offset}" rpy="${right_arm_shoulder_lift_joint_a_offset} ${right_arm_shoulder_lift_joint_b_offset} ${right_arm_shoulder_lift_joint_c_offset}" />
             <parent link="${prefix}shoulder_link" />
             <child link="${prefix}shoulder_lift_offset_link" />
@@ -163,5 +163,5 @@
             <parent link="${prefix}shoulder_lift_offset_link" />
             <child link="${prefix}upper_arm_link" />
-            <origin xyz="0 ${shoulder_offset} 0" rpy="0 ${pi/2.0 + shoulder_lift_joint_offset} 0" />
+            <origin xyz="0 ${shoulder_offset} 0" rpy="0 ${pi/2.0 + right_arm_shoulder_lift_joint_offset} 0" />
             <axis xyz="0 1 0" />
             <calibration rising="0.0" />
@@ -193,5 +193,5 @@
         </link>
         <joint name="${prefix}elbow_offset_joint" type="fixed">
-            <origin xyz="${elbow_joint_x_offset} ${elbow_joint_y_offset} ${elbow_joint_z_offset}" rpy="${elbow_joint_a_offset} ${elbow_joint_b_offset} ${elbow_joint_c_offset}" />
+            <origin xyz="${right_arm_elbow_joint_x_offset} ${right_arm_elbow_joint_y_offset} ${right_arm_elbow_joint_z_offset}" rpy="${right_arm_elbow_joint_a_offset} ${right_arm_elbow_joint_b_offset} ${right_arm_elbow_joint_c_offset}" />
             <parent link="${prefix}upper_arm_link" />
             <child link="${prefix}elbow_offset_link" />
@@ -201,5 +201,5 @@
             <parent link="${prefix}elbow_offset_link" />
             <child link="${prefix}forearm_link" />
-            <origin xyz="0.0 ${elbow_offset} ${upper_arm_length}" rpy="0.0 ${elbow_joint_offset} 0.0" />
+            <origin xyz="0.0 ${elbow_offset} ${upper_arm_length}" rpy="0.0 ${right_arm_elbow_joint_offset} 0.0" />
             <axis xyz="0 1 0" />
             <calibration rising="0.0" />
@@ -231,5 +231,5 @@
         </link>
         <joint name="${prefix}wrist_1_offset_joint" type="fixed">
-            <origin xyz="${wrist_1_joint_x_offset} ${wrist_1_joint_y_offset} ${wrist_1_joint_z_offset}" rpy="${wrist_1_joint_a_offset} ${wrist_1_joint_b_offset} ${wrist_1_joint_c_offset}" />
+            <origin xyz="${right_arm_wrist_1_joint_x_offset} ${right_arm_wrist_1_joint_y_offset} ${right_arm_wrist_1_joint_z_offset}" rpy="${right_arm_wrist_1_joint_a_offset} ${right_arm_wrist_1_joint_b_offset} ${right_arm_wrist_1_joint_c_offset}" />
             <parent link="${prefix}forearm_link" />
             <child link="${prefix}wrist_1_offset_link" />
@@ -239,5 +239,5 @@
             <parent link="${prefix}wrist_1_offset_link" />
             <child link="${prefix}wrist_1_link" />
-            <origin xyz="0 0 ${forearm_length}" rpy="0 ${pi/2.0 + wrist_1_joint_offset} 0" />
+            <origin xyz="0 0 ${forearm_length}" rpy="0 ${pi/2.0 + right_arm_wrist_1_joint_offset} 0" />
             <axis xyz="0 1 0" />
             <calibration rising="0.0" />
@@ -269,5 +269,5 @@
         </link>
         <joint name="${prefix}wrist_2_offset_joint" type="fixed">
-            <origin xyz="${wrist_2_joint_x_offset} ${wrist_2_joint_y_offset} ${wrist_2_joint_z_offset}" rpy="${wrist_2_joint_a_offset} ${wrist_2_joint_b_offset} ${wrist_2_joint_c_offset}" />
+            <origin xyz="${right_arm_wrist_2_joint_x_offset} ${right_arm_wrist_2_joint_y_offset} ${right_arm_wrist_2_joint_z_offset}" rpy="${right_arm_wrist_2_joint_a_offset} ${right_arm_wrist_2_joint_b_offset} ${right_arm_wrist_2_joint_c_offset}" />
             <parent link="${prefix}wrist_1_link" />
             <child link="${prefix}wrist_2_offset_link" />
@@ -277,5 +277,5 @@
             <parent link="${prefix}wrist_2_offset_link" />
             <child link="${prefix}wrist_2_link" />
-            <origin xyz="0.0 ${wrist_1_length} 0.0" rpy="0.0 0.0 ${wrist_2_joint_offset}" />
+            <origin xyz="0.0 ${wrist_1_length} 0.0" rpy="0.0 0.0 ${right_arm_wrist_2_joint_offset}" />
             <axis xyz="0 0 1" />
             <calibration rising="0.0" />
@@ -307,5 +307,5 @@
         </link>
         <joint name="${prefix}wrist_3_offset_joint" type="fixed">
-            <origin xyz="${wrist_3_joint_x_offset} ${wrist_3_joint_y_offset} ${wrist_3_joint_z_offset}" rpy="${wrist_3_joint_a_offset} ${wrist_3_joint_b_offset} ${wrist_3_joint_c_offset}" />
+            <origin xyz="${right_arm_wrist_3_joint_x_offset} ${right_arm_wrist_3_joint_y_offset} ${right_arm_wrist_3_joint_z_offset}" rpy="${right_arm_wrist_3_joint_a_offset} ${right_arm_wrist_3_joint_b_offset} ${right_arm_wrist_3_joint_c_offset}" />
             <parent link="${prefix}wrist_2_link" />
             <child link="${prefix}wrist_3_offset_link" />
@@ -315,5 +315,5 @@
             <parent link="${prefix}wrist_3_offset_link" />
             <child link="${prefix}wrist_3_link" />
-            <origin xyz="0.0 0.0 ${wrist_2_length}" rpy="0.0 ${wrist_3_joint_offset} 0.0" />
+            <origin xyz="0.0 0.0 ${wrist_2_length}" rpy="0.0 ${right_arm_wrist_3_joint_offset} 0.0" />
             <axis xyz="0 1 0" />
             <calibration rising="0.0" />
