Commit message: Added information to extra links to avoid Gazebo errors

File: vulcano_calibrated_ur_description/urdf/calibrated_ur10_vulcano_left_arm.urdf.xacro (robot description, xacro)
@@ -121,5 +121,21 @@
             <child link="${prefix}shoulder_pan_offset_link" />
         </joint>
-        <link name="${prefix}shoulder_pan_offset_link" />
+        <link name="${prefix}shoulder_pan_offset_link">
+          <visual>
+            <geometry>
+              <box size="0.001 0.001 0.001"/>
+            </geometry>
+          </visual>
+          <collision>
+            <geometry>
+              <box size="0.001 0.001 0.001"/>
+            </geometry>
+          </collision>
+          <inertial>
+            <mass value="0.001"/>
+            <origin rpy="0 0 0" xyz="0.0 0.0 0.0"/>
+            <inertia ixx="1e-10" ixy="0.0" ixz="0.0" iyy="1e-10" iyz="0.0" izz="1e-10"/>
+          </inertial>
+        </link>
         <joint name="${prefix}shoulder_pan_joint" type="revolute">
             <parent link="${prefix}shoulder_pan_offset_link" />
@@ -159,5 +175,21 @@
             <child link="${prefix}shoulder_lift_offset_link" />
         </joint>
-        <link name="${prefix}shoulder_lift_offset_link" />
+        <link name="${prefix}shoulder_lift_offset_link">
+          <visual>
+            <geometry>
+              <box size="0.001 0.001 0.001"/>
+            </geometry>
+          </visual>
+          <collision>
+            <geometry>
+              <box size="0.001 0.001 0.001"/>
+            </geometry>
+          </collision>
+          <inertial>
+            <mass value="0.001"/>
+            <origin rpy="0 0 0" xyz="0.0 0.0 0.0"/>
+            <inertia ixx="1e-10" ixy="0.0" ixz="0.0" iyy="1e-10" iyz="0.0" izz="1e-10"/>
+          </inertial>
+        </link>
         <joint name="${prefix}shoulder_lift_joint" type="revolute">
             <parent link="${prefix}shoulder_lift_offset_link" />
@@ -197,5 +229,21 @@
             <child link="${prefix}elbow_offset_link" />
         </joint>
-        <link name="${prefix}elbow_offset_link" />
+        <link name="${prefix}elbow_offset_link">
+          <visual>
+            <geometry>
+              <box size="0.001 0.001 0.001"/>
+            </geometry>
+          </visual>
+          <collision>
+            <geometry>
+              <box size="0.001 0.001 0.001"/>
+            </geometry>
+          </collision>
+          <inertial>
+            <mass value="0.001"/>
+            <origin rpy="0 0 0" xyz="0.0 0.0 0.0"/>
+            <inertia ixx="1e-10" ixy="0.0" ixz="0.0" iyy="1e-10" iyz="0.0" izz="1e-10"/>
+          </inertial>
+        </link>
         <joint name="${prefix}elbow_joint" type="revolute">
             <parent link="${prefix}elbow_offset_link" />
@@ -235,5 +283,21 @@
             <child link="${prefix}wrist_1_offset_link" />
         </joint>
-        <link name="${prefix}wrist_1_offset_link" />
+        <link name="${prefix}wrist_1_offset_link">
+          <visual>
+            <geometry>
+              <box size="0.001 0.001 0.001"/>
+            </geometry>
+          </visual>
+          <collision>
+            <geometry>
+              <box size="0.001 0.001 0.001"/>
+            </geometry>
+          </collision>
+          <inertial>
+            <mass value="0.001"/>
+            <origin rpy="0 0 0" xyz="0.0 0.0 0.0"/>
+            <inertia ixx="1e-10" ixy="0.0" ixz="0.0" iyy="1e-10" iyz="0.0" izz="1e-10"/>
+          </inertial>
+        </link>
         <joint name="${prefix}wrist_1_joint" type="revolute">
             <parent link="${prefix}wrist_1_offset_link" />
@@ -273,5 +337,21 @@
             <child link="${prefix}wrist_2_offset_link" />
         </joint>
-        <link name="${prefix}wrist_2_offset_link" />
+        <link name="${prefix}wrist_2_offset_link">
+          <visual>
+            <geometry>
+              <box size="0.001 0.001 0.001"/>
+            </geometry>
+          </visual>
+          <collision>
+            <geometry>
+              <box size="0.001 0.001 0.001"/>
+            </geometry>
+          </collision>
+          <inertial>
+            <mass value="0.001"/>
+            <origin rpy="0 0 0" xyz="0.0 0.0 0.0"/>
+            <inertia ixx="1e-10" ixy="0.0" ixz="0.0" iyy="1e-10" iyz="0.0" izz="1e-10"/>
+          </inertial>
+        </link>
         <joint name="${prefix}wrist_2_joint" type="revolute">
             <parent link="${prefix}wrist_2_offset_link" />
@@ -311,5 +391,21 @@
             <child link="${prefix}wrist_3_offset_link" />
         </joint>
-        <link name="${prefix}wrist_3_offset_link" />
+        <link name="${prefix}wrist_3_offset_link">
+          <visual>
+            <geometry>
+              <box size="0.001 0.001 0.001"/>
+            </geometry>
+          </visual>
+          <collision>
+            <geometry>
+              <box size="0.001 0.001 0.001"/>
+            </geometry>
+          </collision>
+          <inertial>
+            <mass value="0.001"/>
+            <origin rpy="0 0 0" xyz="0.0 0.0 0.0"/>
+            <inertia ixx="1e-10" ixy="0.0" ixz="0.0" iyy="1e-10" iyz="0.0" izz="1e-10"/>
+          </inertial>
+        </link>
         <joint name="${prefix}wrist_3_joint" type="revolute">
             <parent link="${prefix}wrist_3_offset_link" />

File: vulcano_calibrated_ur_description/urdf/calibrated_ur10_vulcano_right_arm.urdf.xacro (robot description, xacro)
@@ -121,5 +121,21 @@
             <child link="${prefix}shoulder_pan_offset_link" />
         </joint>
-        <link name="${prefix}shoulder_pan_offset_link" />
+        <link name="${prefix}shoulder_pan_offset_link">
+          <visual>
+            <geometry>
+              <box size="0.001 0.001 0.001"/>
+            </geometry>
+          </visual>
+          <collision>
+            <geometry>
+              <box size="0.001 0.001 0.001"/>
+            </geometry>
+          </collision>
+          <inertial>
+            <mass value="0.001"/>
+            <origin rpy="0 0 0" xyz="0.0 0.0 0.0"/>
+            <inertia ixx="1e-10" ixy="0.0" ixz="0.0" iyy="1e-10" iyz="0.0" izz="1e-10"/>
+          </inertial>
+        </link>
         <joint name="${prefix}shoulder_pan_joint" type="revolute">
             <parent link="${prefix}shoulder_pan_offset_link" />
@@ -159,5 +175,21 @@
             <child link="${prefix}shoulder_lift_offset_link" />
         </joint>
-        <link name="${prefix}shoulder_lift_offset_link" />
+        <link name="${prefix}shoulder_lift_offset_link">
+          <visual>
+            <geometry>
+              <box size="0.001 0.001 0.001"/>
+            </geometry>
+          </visual>
+          <collision>
+            <geometry>
+              <box size="0.001 0.001 0.001"/>
+            </geometry>
+          </collision>
+          <inertial>
+            <mass value="0.001"/>
+            <origin rpy="0 0 0" xyz="0.0 0.0 0.0"/>
+            <inertia ixx="1e-10" ixy="0.0" ixz="0.0" iyy="1e-10" iyz="0.0" izz="1e-10"/>
+          </inertial>
+        </link>
         <joint name="${prefix}shoulder_lift_joint" type="revolute">
             <parent link="${prefix}shoulder_lift_offset_link" />
@@ -197,5 +229,21 @@
             <child link="${prefix}elbow_offset_link" />
         </joint>
-        <link name="${prefix}elbow_offset_link" />
+        <link name="${prefix}elbow_offset_link">
+          <visual>
+            <geometry>
+              <box size="0.001 0.001 0.001"/>
+            </geometry>
+          </visual>
+          <collision>
+            <geometry>
+              <box size="0.001 0.001 0.001"/>
+            </geometry>
+          </collision>
+          <inertial>
+            <mass value="0.001"/>
+            <origin rpy="0 0 0" xyz="0.0 0.0 0.0"/>
+            <inertia ixx="1e-10" ixy="0.0" ixz="0.0" iyy="1e-10" iyz="0.0" izz="1e-10"/>
+          </inertial>
+        </link>
         <joint name="${prefix}elbow_joint" type="revolute">
             <parent link="${prefix}elbow_offset_link" />
@@ -235,5 +283,21 @@
             <child link="${prefix}wrist_1_offset_link" />
         </joint>
-        <link name="${prefix}wrist_1_offset_link" />
+        <link name="${prefix}wrist_1_offset_link">
+          <visual>
+            <geometry>
+              <box size="0.001 0.001 0.001"/>
+            </geometry>
+          </visual>
+          <collision>
+            <geometry>
+              <box size="0.001 0.001 0.001"/>
+            </geometry>
+          </collision>
+          <inertial>
+            <mass value="0.001"/>
+            <origin rpy="0 0 0" xyz="0.0 0.0 0.0"/>
+            <inertia ixx="1e-10" ixy="0.0" ixz="0.0" iyy="1e-10" iyz="0.0" izz="1e-10"/>
+          </inertial>
+        </link>
         <joint name="${prefix}wrist_1_joint" type="revolute">
             <parent link="${prefix}wrist_1_offset_link" />
@@ -273,5 +337,21 @@
             <child link="${prefix}wrist_2_offset_link" />
         </joint>
-        <link name="${prefix}wrist_2_offset_link" />
+        <link name="${prefix}wrist_2_offset_link">
+          <visual>
+            <geometry>
+              <box size="0.001 0.001 0.001"/>
+            </geometry>
+          </visual>
+          <collision>
+            <geometry>
+              <box size="0.001 0.001 0.001"/>
+            </geometry>
+          </collision>
+          <inertial>
+            <mass value="0.001"/>
+            <origin rpy="0 0 0" xyz="0.0 0.0 0.0"/>
+            <inertia ixx="1e-10" ixy="0.0" ixz="0.0" iyy="1e-10" iyz="0.0" izz="1e-10"/>
+          </inertial>
+        </link>
         <joint name="${prefix}wrist_2_joint" type="revolute">
             <parent link="${prefix}wrist_2_offset_link" />
@@ -311,5 +391,21 @@
             <child link="${prefix}wrist_3_offset_link" />
         </joint>
-        <link name="${prefix}wrist_3_offset_link" />
+        <link name="${prefix}wrist_3_offset_link">
+          <visual>
+            <geometry>
+              <box size="0.001 0.001 0.001"/>
+            </geometry>
+          </visual>
+          <collision>
+            <geometry>
+              <box size="0.001 0.001 0.001"/>
+            </geometry>
+          </collision>
+          <inertial>
+            <mass value="0.001"/>
+            <origin rpy="0 0 0" xyz="0.0 0.0 0.0"/>
+            <inertia ixx="1e-10" ixy="0.0" ixz="0.0" iyy="1e-10" iyz="0.0" izz="1e-10"/>
+          </inertial>
+        </link>
         <joint name="${prefix}wrist_3_joint" type="revolute">
             <parent link="${prefix}wrist_3_offset_link" />
@@ -357,6 +453,6 @@
             </collision>
         </link>
-        <xacro:ur_arm_transmission prefix="${prefix}" />
-        <xacro:ur_arm_gazebo prefix="${prefix}" />
+        <xacro:calibrated_ur_arm_transmission prefix="${prefix}" />
+        <xacro:calibrated_ur_arm_gazebo prefix="${prefix}" />
         <!-- ROS base_link to UR 'Base' Coordinates transform -->
         <link name="${prefix}base" />

Commit message: Modified calibrated UR's URDF joint limits in wrists

File: vulcano_calibrated_ur_description/urdf/calibrated_ur10_vulcano_left_arm.urdf.xacro (robot description, xacro)
@@ -97,5 +97,6 @@
     <xacro:property name="left_arm_wrist_3_joint_b_offset" value="0.000358152" />
     <xacro:property name="left_arm_wrist_3_joint_c_offset" value="0.00527917" />
-    <xacro:macro name="left_arm_ur10_robot" params="prefix joint_limited shoulder_pan_lower_limit:=${-pi} shoulder_pan_upper_limit:=${pi} shoulder_lift_lower_limit:=${-pi} shoulder_lift_upper_limit:=${pi} elbow_joint_lower_limit:=${-pi} elbow_joint_upper_limit:=${pi} wrist_1_lower_limit:=${-pi} wrist_1_upper_limit:=${pi} wrist_2_lower_limit:=${-pi} wrist_2_upper_limit:=${pi} wrist_3_lower_limit:=${-pi} wrist_3_upper_limit:=${pi}">
+    <!--xacro:macro name="left_arm_ur10_robot" params="prefix joint_limited shoulder_pan_lower_limit:=${-pi} shoulder_pan_upper_limit:=${pi} shoulder_lift_lower_limit:=${-pi} shoulder_lift_upper_limit:=${pi} elbow_joint_lower_limit:=${-pi} elbow_joint_upper_limit:=${pi} wrist_1_lower_limit:=${-pi} wrist_1_upper_limit:=${pi} wrist_2_lower_limit:=${-pi} wrist_2_upper_limit:=${pi} wrist_3_lower_limit:=${-pi} wrist_3_upper_limit:=${pi}"-->
+	<xacro:macro name="left_arm_ur10_robot" params="prefix joint_limited shoulder_pan_lower_limit:=${-pi} shoulder_pan_upper_limit:=${pi} shoulder_lift_lower_limit:=${-pi} shoulder_lift_upper_limit:=${pi} elbow_joint_lower_limit:=${-pi} elbow_joint_upper_limit:=${pi} wrist_1_lower_limit:=${-2*pi} wrist_1_upper_limit:=${2*pi} wrist_2_lower_limit:=${-2*pi} wrist_2_upper_limit:=${2*pi} wrist_3_lower_limit:=${-2*pi} wrist_3_upper_limit:=${2*pi}">
         <link name="${prefix}base_link">
             <visual>

File: vulcano_calibrated_ur_description/urdf/calibrated_ur10_vulcano_right_arm.urdf.xacro (robot description, xacro)
@@ -97,5 +97,6 @@
     <xacro:property name="right_arm_wrist_3_joint_b_offset" value="-0.000202165" />
     <xacro:property name="right_arm_wrist_3_joint_c_offset" value="0.000150637" />
-    <xacro:macro name="right_arm_ur10_robot" params="prefix joint_limited shoulder_pan_lower_limit:=${-pi} shoulder_pan_upper_limit:=${pi} shoulder_lift_lower_limit:=${-pi} shoulder_lift_upper_limit:=${pi} elbow_joint_lower_limit:=${-pi} elbow_joint_upper_limit:=${pi} wrist_1_lower_limit:=${-pi} wrist_1_upper_limit:=${pi} wrist_2_lower_limit:=${-pi} wrist_2_upper_limit:=${pi} wrist_3_lower_limit:=${-pi} wrist_3_upper_limit:=${pi}">
+    <!--xacro:macro name="right_arm_ur10_robot" params="prefix joint_limited shoulder_pan_lower_limit:=${-pi} shoulder_pan_upper_limit:=${pi} shoulder_lift_lower_limit:=${-pi} shoulder_lift_upper_limit:=${pi} elbow_joint_lower_limit:=${-pi} elbow_joint_upper_limit:=${pi} wrist_1_lower_limit:=${-pi} wrist_1_upper_limit:=${pi} wrist_2_lower_limit:=${-pi} wrist_2_upper_limit:=${pi} wrist_3_lower_limit:=${-pi} wrist_3_upper_limit:=${pi}"-->
+	<xacro:macro name="right_arm_ur10_robot" params="prefix joint_limited shoulder_pan_lower_limit:=${-pi} shoulder_pan_upper_limit:=${pi} shoulder_lift_lower_limit:=${-pi} shoulder_lift_upper_limit:=${pi} elbow_joint_lower_limit:=${-pi} elbow_joint_upper_limit:=${pi} wrist_1_lower_limit:=${-2*pi} wrist_1_upper_limit:=${2*pi} wrist_2_lower_limit:=${-2*pi} wrist_2_upper_limit:=${2*pi} wrist_3_lower_limit:=${-2*pi} wrist_3_upper_limit:=${2*pi}">
         <link name="${prefix}base_link">
             <visual>
