Commit message: Corrected masses of torso

File: vulcano_torso_description/urdf/vulcano_torso.urdf.xacro (robot description, xacro)
@@ -10,5 +10,5 @@
       <inertial>
         <origin xyz="0 0 0" rpy="0 0 0 "/>
-        <mass value="1000"/>
+        <mass value="5"/> <!-- TODO: check masses -->
         <inertia ixx="1.0" ixy="0.0" ixz="0.0" iyy="1.0" iyz="0.0" izz="1.0"/>
       </inertial>
@@ -39,5 +39,5 @@
       <inertial>
         <origin xyz="0 0 0" rpy="0 0 0"/>
-        <mass value="1000"/>
+        <mass value="5"/>
         <inertia ixx="1.0" ixy="0.0" ixz="0.0" iyy="1.0" iyz="0.0" izz="1.0"/>
       </inertial>
@@ -71,5 +71,5 @@
       <inertial>
         <origin xyz="0 0 0" rpy="0 0 0"/>
-        <mass value="1000"/>
+        <mass value="5"/>
         <inertia ixx="1.0" ixy="0.0" ixz="0.0" iyy="1.0" iyz="0.0" izz="1.0"/>
       </inertial>

Commit message: Vulcano torso URDF modified to correct Kinect optical frame (torso calibration [0.650,0,0,0])

File: vulcano_torso_description/urdf/vulcano_torso.urdf.xacro (robot description, xacro)
@@ -10,5 +10,6 @@
     <xacro:include filename="$(find vulcano_torso_description)/urdf/pantilt/pantilt.urdf.xacro"/>
     <xacro:include filename="$(find vulcano_torso_description)/urdf/tube_support/tube_support.urdf.xacro"/>
-    <xacro:include filename="$(find robotnik_sensors)/urdf/all_sensors.urdf.xacro" />
+    <!--xacro:include filename="$(find robotnik_sensors)/urdf/all_sensors.urdf.xacro" /-->
+    <xacro:include filename="$(find vulcano_torso_description)/urdf/pantilt/kinectv2.urdf.xacro" />
     <xacro:macro name="vulcano_torso" params="prefix hq"> <!-- TODO: check hq variable -->
         <link name="${prefix}torso_base_link">
@@ -33,5 +34,20 @@
             </inertial>
         </link>
-        <xacro:pantilt prefix="${prefix}" parent="${prefix}torso_guidance_pantilt_link" hq="${hq}"/>
+        <!-- CALIBRATION OFFSET -->
+        <joint name="${prefix}pantilt_offset_joint" type="fixed">
+          <origin xyz="0.03506 -0.01853 -0.00396" rpy="3.12736 -3.10935 3.13263"/>
+          <parent link="${prefix}torso_guidance_pantilt_link"/>
+          <child link="${prefix}pantilt_offset_link"/>
+          <axis xyz="0 0 1"/>
+        </joint>
+        <link name="${prefix}pantilt_offset_link">
+            <inertial>
+                <origin xyz="0 0 0" rpy="0 0 0 "/>
+                <mass value="0"/>
+            <inertia ixx="1.0" ixy="0.0" ixz="0.0" iyy="1.0" iyz="0.0" izz="1.0"/>
+            </inertial>
+        </link>
+        <xacro:pantilt prefix="${prefix}" parent="${prefix}pantilt_offset_link" hq="${hq}"/>
+        <!--xacro:pantilt prefix="${prefix}" parent="${prefix}torso_guidance_pantilt_link" hq="${hq}"/-->
         <!-- TODO: check kinect2 position -->
         <xacro:sensor_kinectv2 name="${prefix}torso_kinect" parent="${prefix}torso_pantilt_link" base="true">
