Commit message: vulcano_pantilt: added pantilt controllers

File: vulcano_torso_description/urdf/pantilt/pantilt.urdf.xacro (robot description, xacro)
@@ -69,5 +69,5 @@
       <child link="${prefix}torso_pantilt_pan_link"/>
       <axis xyz="0 0 1"/>
-      <limit lower="${-180*deg2rad}" upper="${180*deg2rad}" effort="100" velocity="100"/>
+      <limit lower="${-55*deg2rad}" upper="${55*deg2rad}" effort="100" velocity="100"/>
       <dynamics friction="1000" damping="1000"/>
     </joint>
@@ -75,10 +75,9 @@
       <type>transmission_interface/SimpleTransmission</type>
       <joint name="${prefix}torso_pantilt_pan_joint">
-        <!--<hardwareInterface>EffortJointInterface</hardwareInterface>-->
         <hardwareInterface>PositionJointInterface</hardwareInterface><!-- TODO: PositionJointInterface? EffortJointInterface? -->
       </joint>
       <actuator name="${prefix}torso_pantilt_pan_motor">
         <mechanicalReduction>1</mechanicalReduction>
-        <hardwareInterface>EffortJointInterface</hardwareInterface>
+        <hardwareInterface>PositionJointInterface</hardwareInterface>
       </actuator>
     </transmission>
@@ -111,5 +110,5 @@
       <child link="${prefix}torso_pantilt_tilt_base_link"/>
       <axis xyz="0 0 1"/>
-      <limit lower="${-180*deg2rad}" upper="${180*deg2rad}" effort="100" velocity="100"/>
+      <limit lower="${-70*deg2rad}" upper="${40*deg2rad}" effort="100" velocity="100"/>
       <dynamics friction="1000" damping="1000"/>
     </joint>
@@ -122,5 +121,5 @@
       <actuator name="${prefix}torso_pantilt_tilt_motor">
         <mechanicalReduction>1</mechanicalReduction>
-        <hardwareInterface>EffortJointInterface</hardwareInterface>
+        <hardwareInterface>PositionJointInterface</hardwareInterface>
       </actuator>
     </transmission>

Commit message: vulcano_torso_description: corrected tilt limits

File: vulcano_torso_description/urdf/pantilt/pantilt.urdf.xacro (robot description, xacro)
@@ -110,5 +110,5 @@
       <child link="${prefix}torso_pantilt_tilt_base_link"/>
       <axis xyz="0 0 1"/>
-      <limit lower="${-70*deg2rad}" upper="${40*deg2rad}" effort="100" velocity="100"/>
+      <limit lower="${-40*deg2rad}" upper="${70*deg2rad}" effort="100" velocity="100"/>
       <dynamics friction="1000" damping="1000"/>
     </joint>

Commit message: torso_description: switch name to prefix param

File: vulcano_torso_description/urdf/pantilt/pantilt.urdf.xacro (robot description, xacro)
@@ -110,5 +110,5 @@
       <child link="${prefix}torso_pantilt_tilt_base_link"/>
       <axis xyz="0 0 1"/>
-      <limit lower="${-40*deg2rad}" upper="${70*deg2rad}" effort="100" velocity="100"/>
+      <limit lower="${-360*deg2rad}" upper="${360*deg2rad}" effort="100" velocity="100"/>
       <dynamics friction="1000" damping="1000"/>
     </joint>

File: vulcano_torso_description/urdf/vulcano_torso.urdf.xacro (robot description, xacro)
@@ -35,11 +35,11 @@
         <xacro:pantilt prefix="${prefix}" parent="${prefix}torso_guidance_pantilt_link" hq="${hq}"/>
         <!-- TODO: check kinect2 position -->
-        <xacro:sensor_kinectv2 name="${prefix}torso_kinect" parent="${prefix}torso_pantilt_link" base="true">
+        <xacro:sensor_kinectv2 prefix="${prefix}torso_kinect" parent="${prefix}torso_pantilt_link" base="true">
             <origin xyz="0.01255 0 0.066" rpy="0 0 0"/>
         </xacro:sensor_kinectv2>
-        <xacro:sensor_ueye_cp_gige name="${prefix}torso_ueye_left" parent="${prefix}torso_pantilt_link">
+        <xacro:sensor_ueye_cp_gige prefix="${prefix}torso_ueye_left" parent="${prefix}torso_pantilt_link">
             <origin xyz="0.0258 -0.14975 0.0165" rpy="0 0 0"/>
         </xacro:sensor_ueye_cp_gige>
-        <xacro:sensor_ueye_cp_gige name="${prefix}torso_ueye_right" parent="${prefix}torso_pantilt_link">
+        <xacro:sensor_ueye_cp_gige prefix="${prefix}torso_ueye_right" parent="${prefix}torso_pantilt_link">
             <origin xyz="0.0258 0.14975 0.0165" rpy="0 0 0"/>
         </xacro:sensor_ueye_cp_gige>

Commit message: torso_description: updated pantilt joint limits

File: vulcano_torso_description/urdf/pantilt/pantilt.urdf.xacro (robot description, xacro)
@@ -2,5 +2,4 @@
 <robot xmlns:xacro="http://ros.org/wiki/xacro">
   <xacro:property name="PI" value="3.1415926535897931"/>
-  <xacro:property name="deg2rad" value="0.01745329251"/>
   <!-- Define the torso -->
   <xacro:macro name="pantilt" params="prefix parent hq">
@@ -69,5 +68,5 @@
       <child link="${prefix}torso_pantilt_pan_link"/>
       <axis xyz="0 0 1"/>
-      <limit lower="${-55*deg2rad}" upper="${55*deg2rad}" effort="100" velocity="100"/>
+      <limit lower="-0.95" upper="0.95" effort="100" velocity="100"/>
       <dynamics friction="1000" damping="1000"/>
     </joint>
@@ -106,9 +105,9 @@
     <!-- TILT JOINT/LINK -->
     <joint name="${prefix}torso_pantilt_tilt_joint" type="revolute">
-      <origin xyz="0.0 -0.027 0.0" rpy="${-90*deg2rad} 0 0"/>
+      <origin xyz="0.0 -0.027 0.0" rpy="-1.57 0 0"/>
       <parent link="${prefix}torso_pantilt_pan_link"/>
       <child link="${prefix}torso_pantilt_tilt_base_link"/>
       <axis xyz="0 0 1"/>
-      <limit lower="${-360*deg2rad}" upper="${360*deg2rad}" effort="100" velocity="100"/>
+      <limit lower="-1.26" upper="1.26" effort="100" velocity="100"/>
       <dynamics friction="1000" damping="1000"/>
     </joint>
@@ -147,5 +146,5 @@
     </link>
     <joint name="${prefix}torso_pantilt_tilt_support_joint" type="fixed">
-      <origin xyz="0.0 0.0 0.0" rpy="${90*deg2rad} 0 0"/>
+      <origin xyz="0.0 0.0 0.0" rpy="1.57 0 0"/>
       <parent link="${prefix}torso_pantilt_tilt_base_link"/>
       <child link="${prefix}torso_pantilt_tilt_support_link"/>
@@ -176,5 +175,5 @@
     <joint name="${prefix}torso_pantilt_tilt_fixed_joint" type="fixed">
       <!--<origin xyz="0.0 0.027 0.027" rpy="0 0 0"/>-->
-      <origin xyz="0.0 -0.027 0.027" rpy="${90*deg2rad} 0 0"/>
+      <origin xyz="0.0 -0.027 0.027" rpy="1.57 0 0"/>
       <parent link="${prefix}torso_pantilt_tilt_base_link"/>
       <child link="${prefix}torso_pantilt_tilt_link"/>
