Commit message: description: updated model

File: vulcano_base_description/urdf/bases/base.gazebo.xacro (robot description, xacro)
@@ -1,36 +1,4 @@
 <?xml version="1.0"?>
 <robot xmlns:xacro="http://ros.org/wiki/xacro">
-  <xacro:macro name="omni_steering">
-		<gazebo>
-	    <plugin name="omni_steering" filename="libgazebo_ros_planar_move.so">
-		  <robotNamespace>/vulcano_base</robotNamespace>
-	      <commandTopic>/vulcano_base_control/cmd_vel</commandTopic>
-	      <odometryTopic>/vulcano_base/odom</odometryTopic>
-	      <odometryFrame>odom</odometryFrame>
-	      <odometryRate>20.0</odometryRate>
-	      <robotBaseFrame>base_footprint</robotBaseFrame>
-	    </plugin>
-	  </gazebo>
-  </xacro:macro>
-  <xacro:macro name="omni_drive">
-		<gazebo>
-		<plugin name="omni_drive" filename="libomnidrive_plugin.so">
-			<!--<robotNamespace>/vulcano_base</robotNamespace>-->
-			<!--<robotParam>robot_description</robotParam>-->
-			<broadcastTF>1</broadcastTF>
-			<wheelDiameter>0.15</wheelDiameter>
-			<wheelBase>0.933</wheelBase>
-			<trackWidth>0.57</trackWidth>
-			<wheelTorque>40.0</wheelTorque>
-			<motorWheelTorque>25.0</motorWheelTorque>
-			<commandTopic>cmd_vel</commandTopic>  <!-- TODO: review topics -->
-			<odometryTopic>odom</odometryTopic>
-			<odometryFrame>odom</odometryFrame>
-			<odometrySource>encoder</odometrySource>
-			<robotBaseFrame>base_footprint</robotBaseFrame>
-			<updateRate>100.0</updateRate>
-		</plugin>
-		</gazebo>
-  </xacro:macro>
   <gazebo reference="base_footprint">
     <material>Gazebo/Green</material>

File: vulcano_base_description/urdf/bases/base.urdf.xacro (robot description, xacro)
@@ -5,4 +5,9 @@
   <xacro:property name="PI" value="3.1415926535897931"/>
   <xacro:property name="wheel_width" value="0.075" />
+  <xacro:macro name="box_inertia" params="m x y z">
+    <inertia  ixx="${m*(y*y+z*z)/12}" ixy = "0" ixz = "0"
+              iyy="${m*(x*x+z*z)/12}" iyz = "0"
+              izz="${m*(x*x+y*y)/12}" />
+  </xacro:macro>
   <!-- BASE FOOTPRINT -->
   <xacro:if value="${publish_bf}">
@@ -23,9 +28,9 @@
   <!-- BASE_LINK -->
   <link name="${prefix}base_link">
-    <!--<inertial>-->
-      <!--<mass value="184.0" />-->
-      <!--<origin xyz="-0.004 0 -0.357" />-->
-      <!--<inertia  ixx="13.113" ixy="0.131"  ixz="-0.010"  iyy="30.242"  iyz="0.0"  izz="41.3630" />-->
-    <!--</inertial>-->
+     <inertial>
+        <mass value="1000" />
+        <origin xyz="0 0 0" />
+        <box_inertia m="1000" x="0.7" y="0.4" z="0.2"/>
+      </inertial>
     <visual>
        <origin xyz="0 0 0" rpy="0 0 0" />

File: vulcano_base_description/urdf/vulcano_base.urdf.xacro (robot description, xacro)
@@ -29,14 +29,14 @@
     <xacro:macro name="vulcano_base" params="prefix publish_bf hq">
         <xacro:base prefix="${prefix}" publish_bf="${publish_bf}" hq="${hq}"/>
-        <xacro:motor_wheel prefix="${prefix}front_right_" parent="${prefix}base_link" reflect="false" hq="true">
+        <xacro:motor_wheel prefix="${prefix}front_right_" parent="${prefix}base_link" hq="true">
           <origin xyz="${wheel_offset_x} -${wheel_offset_y} ${wheel_offset_z}" rpy="0 0 0"/>
         </xacro:motor_wheel>
-        <xacro:motor_wheel prefix="${prefix}front_left_" parent="${prefix}base_link" reflect="false" hq="true">
+        <xacro:motor_wheel prefix="${prefix}front_left_" parent="${prefix}base_link" hq="true">
           <origin xyz="${wheel_offset_x} ${wheel_offset_y} ${wheel_offset_z}" rpy="0 0 ${180.0*deg2rad}"/>
         </xacro:motor_wheel>
-        <xacro:motor_wheel prefix="${prefix}back_left_" parent="${prefix}base_link" reflect="false" hq="true">
+        <xacro:motor_wheel prefix="${prefix}back_left_" parent="${prefix}base_link" hq="true">
           <origin xyz="-${wheel_offset_x} ${wheel_offset_y} ${wheel_offset_z}" rpy="0 0 ${180.0*deg2rad}"/>
         </xacro:motor_wheel>
-        <xacro:motor_wheel prefix="${prefix}back_right_" parent="${prefix}base_link" reflect="false" hq="true">
+        <xacro:motor_wheel prefix="${prefix}back_right_" parent="${prefix}base_link" hq="true">
           <origin xyz="-${wheel_offset_x} -${wheel_offset_y} ${wheel_offset_z}" rpy="0 0 0"/>
         </xacro:motor_wheel>

File: vulcano_base_description/urdf/wheels/motor_wheel.urdf.xacro (robot description, xacro)
@@ -6,12 +6,12 @@
   <xacro:property name="wheel_height" value="0.14" />
   <xacro:property name="wheel_mass" value="5.0" /> <!-- in kg-->
-  <xacro:property name="steer_joint_damping" value="2.0" />
-  <xacro:property name="steer_joint_friction" value="1.0" />
+  <xacro:property name="steer_joint_damping" value="2000.0" />
+  <xacro:property name="steer_joint_friction" value="1000.0" />
   <xacro:property name="steer_joint_effort_limit" value="100.0" />
   <xacro:property name="steer_joint_velocity_limit" value="2" />
   <xacro:property name="steer_joint_position_limit" value="2.9" />
   <xacro:property name="steer_mechanical_reduction" value="1.0" />
-  <xacro:property name="traction_joint_damping" value="0.001" />
-  <xacro:property name="traction_joint_friction" value="0.001" />
+  <xacro:property name="traction_joint_damping" value="1000.0" />
+  <xacro:property name="traction_joint_friction" value="1000.0" />
   <xacro:property name="traction_joint_effort_limit" value="1000.0" />
   <xacro:property name="traction_joint_velocity_limit" value="6.28" />
@@ -22,6 +22,5 @@
               izz="${m*r*r/2}" />
   </xacro:macro>
-  <xacro:macro name="motor_wheel" params="prefix parent *origin reflect hq">
-  <!-- TODO: check reflect parameter -->
+  <xacro:macro name="motor_wheel" params="prefix parent *origin hq">
   <!--MOTOR WHEEL -->
     <joint name="${prefix}wheel_steer_joint" type="revolute">
@@ -31,5 +30,5 @@
       <axis xyz="0 0 1" rpy="0 0 0" />
       <limit effort="${steer_joint_effort_limit}" velocity="${steer_joint_velocity_limit}" lower="-${steer_joint_position_limit}" upper="${steer_joint_position_limit}"/>
-      <joint_properties damping="${steer_joint_damping}" friction="${steer_joint_friction}"/>
+      <dynamics damping="${steer_joint_damping}" friction="${steer_joint_friction}"/>
     </joint>
   <transmission name="${prefix}wheel_steer_trans">
@@ -49,10 +48,5 @@
           <origin xyz="0 0 0" rpy="0 0 0" />
           <geometry>
-                <xacro:if value="${reflect}">
-                    <mesh filename="package://vulcano_base_description/meshes/wheels/hub.stl" />
-                </xacro:if>
-                <xacro:unless value="${reflect}">
-                    <mesh filename="package://vulcano_base_description/meshes/wheels/hub.stl" />
-                </xacro:unless>
+                <mesh filename="package://vulcano_base_description/meshes/wheels/hub.stl" />
           </geometry>
         </xacro:if>
@@ -61,10 +55,5 @@
           <origin xyz="0 0 0" rpy="0 0 0" />
           <geometry>
-                <xacro:if value="${reflect}">
-                    <mesh filename="package://vulcano_base_description/meshes/wheels/hub.stl" />
-                </xacro:if>
-                <xacro:unless value="${reflect}">
-                    <mesh filename="package://vulcano_base_description/meshes/wheels/hub.stl" />
-                </xacro:unless>
+                <mesh filename="package://vulcano_base_description/meshes/wheels/hub.stl" />
           </geometry>
         </xacro:unless>
@@ -73,16 +62,11 @@
         <origin xyz="0 0 0" rpy="0 0 0" />
         <geometry>
-                <xacro:if value="${reflect}">
-                    <mesh filename="package://vulcano_base_description/meshes/wheels/hub.stl" />
-                </xacro:if>
-                <xacro:unless value="${reflect}">
-                    <mesh filename="package://vulcano_base_description/meshes/wheels/hub.stl" />
-                </xacro:unless>
+             <mesh filename="package://vulcano_base_description/meshes/wheels/hub.stl" />
         </geometry>
       </collision>
       <inertial>
-        <mass value="10" />
+        <mass value="${wheel_mass}" />
         <origin xyz="0 0 0" />
-        <inertia  ixx="0.01" ixy="0.0"  ixz="0.0"  iyy="0.01"  iyz="0.0"  izz="0.01" />
+        <cylinder_inertia  m="${wheel_mass}" r="${wheel_height}" h="${wheel_radius}" /> <!-- TODO: check inertia -->
       </inertial>
     </link>
@@ -94,5 +78,5 @@
         <axis xyz="0 1 0" rpy="0 0 0" />
         <limit effort="${traction_joint_effort_limit}" velocity="${traction_joint_velocity_limit}"/>
-        <joint_properties damping="${traction_joint_damping}" friction="{traction_joint_friction}"/>
+        <dynamics damping="${traction_joint_damping}" friction="${traction_joint_friction}"/>
     </joint>
     <transmission name="${prefix}wheel_traction">
@@ -112,31 +96,18 @@
           <origin xyz="0 0 0" rpy="0 0 0" />
           <geometry>
-                <xacro:if value="${reflect}">
-                    <mesh filename="package://vulcano_base_description/meshes/wheels/rubber_band.stl" />
-                </xacro:if>
-                <xacro:unless value="${reflect}">
-                    <mesh filename="package://vulcano_base_description/meshes/wheels/rubber_band.stl" />
-                </xacro:unless>
+              <mesh filename="package://vulcano_base_description/meshes/wheels/rubber_band.stl" />
           </geometry>
         </xacro:if>
        <!-- LOW RESOLUTION WHEELS -->
         <xacro:unless value="${hq}">
-          <origin xyz="0 0 0" rpy="${M_PI/2} 0 0" />
+          <origin xyz="0 0 0" rpy="0 0 0" />
           <geometry>
-            <cylinder length="${wheel_height}" radius="${wheel_radius}" />
+              <mesh filename="package://vulcano_base_description/meshes/wheels/rubber_band.stl" />
           </geometry>
         </xacro:unless>
       </visual>
       <collision>
-        <origin xyz="0 0 0" rpy="${M_PI/2} 0 0" />
+        <origin xyz="0 0 0" rpy="0 0 0" />
         <geometry>
-          <!--<xacro:if value="${reflect}">-->
-              <!--<mesh filename="package://vulcano_base_description/meshes/wheels/wheel_1.dae" />-->
-          <!--</xacro:if>-->
-          <!--<xacro:unless value="${reflect}">-->
-              <!--<mesh filename="package://vulcano_base_description/meshes/wheels/wheel_1.dae" />-->
-          <!--</xacro:unless>-->
-          <!-- cylinder length="${wheel_height}" radius="${wheel_radius}" / -->
-          <!--sphere radius="${wheel_radius}" /-->
           <mesh filename="package://vulcano_base_description/meshes/wheels/rubber_band.stl" />
         </geometry>
@@ -148,4 +119,12 @@
       </inertial>
    </link>
+   <!--<gazebo reference="${prefix}wheel_tracion_link">-->
+        <!--<mu1 value="1.0"/>-->
+        <!--<mu2 value="1.0"/>-->
+        <!--[><kp value="10000000.0" /><]-->
+        <!--[><kd value="1.0" /><]-->
+        <!--[><fdir1 value="1 0 0"/><]-->
+        <!--[><turnGravityOff>false</turnGravityOff><]-->
+   <!--</gazebo>-->
    <!-- gazebo reference="${prefix}motor_wheel_link">
         <mu1 value="1.0"/>
