Commit message: base_description: ported from indigo-devel

File: vulcano_base_description/urdf/bases/base.gazebo.xacro (robot description, xacro)
@@ -1,4 +1,36 @@
 <?xml version="1.0"?>
 <robot xmlns:xacro="http://ros.org/wiki/xacro">
+  <xacro:macro name="omni_steering">
+		<gazebo>
+	    <plugin name="omni_steering" filename="libgazebo_ros_planar_move.so">
+		  <robotNamespace>/vulcano_base</robotNamespace>
+	      <commandTopic>/vulcano_base_control/cmd_vel</commandTopic>
+	      <odometryTopic>/vulcano_base/odom</odometryTopic>
+	      <odometryFrame>odom</odometryFrame>
+	      <odometryRate>20.0</odometryRate>
+	      <robotBaseFrame>base_footprint</robotBaseFrame>
+	    </plugin>
+	  </gazebo>
+  </xacro:macro>
+  <xacro:macro name="omni_drive">
+		<gazebo>
+		<plugin name="omni_drive" filename="libomnidrive_plugin.so">
+			<!--<robotNamespace>/vulcano_base</robotNamespace>-->
+			<!--<robotParam>robot_description</robotParam>-->
+			<broadcastTF>1</broadcastTF>
+			<wheelDiameter>0.15</wheelDiameter>
+			<wheelBase>0.933</wheelBase>
+			<trackWidth>0.57</trackWidth>
+			<wheelTorque>40.0</wheelTorque>
+			<motorWheelTorque>25.0</motorWheelTorque>
+			<commandTopic>cmd_vel</commandTopic>  <!-- TODO: review topics -->
+			<odometryTopic>odom</odometryTopic>
+			<odometryFrame>odom</odometryFrame>
+			<odometrySource>encoder</odometrySource>
+			<robotBaseFrame>base_footprint</robotBaseFrame>
+			<updateRate>100.0</updateRate>
+		</plugin>
+		</gazebo>
+  </xacro:macro>
   <gazebo reference="base_footprint">
     <material>Gazebo/Green</material>

File: vulcano_base_description/urdf/bases/base.urdf.xacro (robot description, xacro)
@@ -5,9 +5,4 @@
   <xacro:property name="PI" value="3.1415926535897931"/>
   <xacro:property name="wheel_width" value="0.075" />
-  <xacro:macro name="box_inertia" params="m x y z">
-    <inertia  ixx="${m*(y*y+z*z)/12}" ixy = "0" ixz = "0"
-              iyy="${m*(x*x+z*z)/12}" iyz = "0"
-              izz="${m*(x*x+y*y)/12}" />
-  </xacro:macro>
   <!-- BASE FOOTPRINT -->
   <xacro:if value="${publish_bf}">
@@ -20,5 +15,5 @@
       </visual>
     </link>
-    <joint name="${prefix}base_footprint_joint" type="fixed">
+    <joint name="base_footprint_joint" type="fixed">
       <origin xyz="0 0 ${wheel_radius}" rpy="0 0 0" /> <!-- ${wheel_radius} property must be defined inside wheel description -->
       <parent link="${prefix}base_footprint"/>
@@ -28,16 +23,21 @@
   <!-- BASE_LINK -->
   <link name="${prefix}base_link">
-     <inertial>
-        <mass value="1000" />
-        <origin xyz="0 0 0" />
-        <box_inertia m="1000" x="0.7" y="0.4" z="0.2"/>
-      </inertial>
+    <inertial>
+      <mass value="184.0" />
+      <origin xyz="-0.004 0 -0.357" />
+      <inertia  ixx="13.113" ixy="0.131"  ixz="-0.010"  iyy="30.242"  iyz="0.0"  izz="41.3630" />
+    </inertial>
     <visual>
        <origin xyz="0 0 0" rpy="0 0 0" />
-       <!--<xacro:if value="${hq}">-->
+       <xacro:if value="${hq}">
        <geometry>
-	     <mesh filename="package://vulcano_base_description/meshes/bases/cabinet.stl"/>
+	     <mesh filename="package://vulcano_base_description/meshes/bases/vulcano_base_chassis.dae"/>
        </geometry>
-       <!--</xacro:if>-->
+       </xacro:if>
+       <xacro:unless value="${hq}">
+       <geometry>
+	     <mesh filename="package://vulcano_base_description/meshes/bases/vulcano_base_chassis.dae"/>
+       </geometry>
+       </xacro:unless>
        <material name="darkgrey">
          <color rgba="0.1 0.1 0.1 1"/>
@@ -47,8 +47,42 @@
        <origin xyz="0 0 0" rpy="0 0 0 " />
        <geometry>
-	     <mesh filename="package://vulcano_base_description/meshes/bases/cabinet.stl"/>
+         <mesh filename="package://vulcano_base_description/meshes/bases/vulcano_base_chassis.dae"/>
        </geometry>
     </collision>
   </link>
+  <link name="${prefix}cabinet_link">
+    <inertial>
+      <mass value="96.0" />
+      <origin xyz="-0.089 -0.001 0.00417" />
+      <inertia  ixx="10.783" ixy="-0.137"  ixz="-1.976"  iyy="18.311"  iyz="0.042"  izz="19.866" />
+    </inertial>
+    <visual>
+       <origin xyz="0 0 0" rpy="0 0 0" />
+       <xacro:if value="${hq}">
+       <geometry>
+	     <mesh filename="package://vulcano_base_description/meshes/bases/vulcano_base_cabinet.dae"/>
+       </geometry>
+       </xacro:if>
+       <xacro:unless value="${hq}">
+       <geometry>
+	     <mesh filename="package://vulcano_base_description/meshes/bases/vulcano_base_cabinet.dae"/>
+       </geometry>
+       </xacro:unless>
+       <material name="darkgrey">
+         <color rgba="0.1 0.1 0.1 1"/>
+       </material>
+    </visual>
+    <collision>
+       <origin xyz="0 0 0" rpy="0 0 0 " />
+       <geometry>
+         <mesh filename="package://vulcano_base_description/meshes/bases/vulcano_base_cabinet.dae"/>
+       </geometry>
+    </collision>
+  </link>
+  <joint name="${prefix}cabinet_joint" type="fixed">
+    <origin xyz="0 0 0.234" rpy="0 0 0" />
+    <parent link="${prefix}base_link"/>
+    <child link="${prefix}cabinet_link" />
+  </joint>
   </xacro:macro>
 </robot>

File: vulcano_base_description/urdf/vulcano_base.urdf.xacro (robot description, xacro)
@@ -15,9 +15,8 @@
     <!-- Global parameters -->
     <!-- ***************** -->
-    <xacro:property name="vulcano_base_version" value="2.0" />    <!-- x,y,z in translation from base_link to the center of the wheel -->
     <xacro:property name="PI" value="3.1415926535897931"/>
     <xacro:property name="deg2rad" value="0.01745329251"/>
     <!-- Wheel parameters -->
-    <xacro:property name="wheel_offset_x" value="0.6165" />    <!-- x,y,z in translation from base_link to the center of the wheel -->
+    <xacro:property name="wheel_offset_x" value="0.467" />    <!-- x,y,z in translation from base_link to the center of the wheel -->
     <xacro:property name="wheel_offset_y" value="0.285" />
     <xacro:property name="wheel_offset_z" value="0.0" />
@@ -29,26 +28,32 @@
     <xacro:macro name="vulcano_base" params="prefix publish_bf hq">
         <xacro:base prefix="${prefix}" publish_bf="${publish_bf}" hq="${hq}"/>
-        <xacro:motor_wheel prefix="${prefix}front_right_" parent="${prefix}base_link" hq="true">
+        <xacro:motor_wheel prefix="${prefix}front_right_" parent="${prefix}base_link" reflect="false" hq="true">
           <origin xyz="${wheel_offset_x} -${wheel_offset_y} ${wheel_offset_z}" rpy="0 0 0"/>
         </xacro:motor_wheel>
-        <xacro:motor_wheel prefix="${prefix}front_left_" parent="${prefix}base_link" hq="true">
+        <xacro:motor_wheel prefix="${prefix}front_left_" parent="${prefix}base_link" reflect="false" hq="true">
           <origin xyz="${wheel_offset_x} ${wheel_offset_y} ${wheel_offset_z}" rpy="0 0 ${180.0*deg2rad}"/>
         </xacro:motor_wheel>
-        <xacro:motor_wheel prefix="${prefix}back_left_" parent="${prefix}base_link" hq="true">
+        <xacro:motor_wheel prefix="${prefix}back_left_" parent="${prefix}base_link" reflect="false" hq="true">
           <origin xyz="-${wheel_offset_x} ${wheel_offset_y} ${wheel_offset_z}" rpy="0 0 ${180.0*deg2rad}"/>
         </xacro:motor_wheel>
-        <xacro:motor_wheel prefix="${prefix}back_right_" parent="${prefix}base_link" hq="true">
+        <xacro:motor_wheel prefix="${prefix}back_right_" parent="${prefix}base_link" reflect="false" hq="true">
           <origin xyz="-${wheel_offset_x} -${wheel_offset_y} ${wheel_offset_z}" rpy="0 0 0"/>
         </xacro:motor_wheel>
         <!-- SENSORS see robotnik_sensors for the specific configuration -->
-        <xacro:sensor_imu prefix="${prefix}imu" parent="${prefix}base_link">
+        <xacro:sensor_imu name="imu" parent="${prefix}base_link">
           <origin xyz="-0.40 0.06 0.75" rpy="0 0 0"/>
         </xacro:sensor_imu>
-        <xacro:sensor_sick_s300 prefix="${prefix}front_left_laser" parent="${prefix}base_link">
-            <origin xyz="0.75631 0.34581 0.30676" rpy="${180*deg2rad} 0 ${45*deg2rad}"/>
+        <xacro:sensor_sick_s300 name="front_left_laser" parent="${prefix}base_link">
+            <origin xyz="0.606321 0.345821 0.3095" rpy="${180*deg2rad} 0 ${45*deg2rad}"/>
         </xacro:sensor_sick_s300>
-        <xacro:sensor_sick_s300 prefix="${prefix}back_right_laser" parent="${prefix}base_link">
-            <origin xyz="-0.75631 -0.34581 0.30676" rpy="${180*deg2rad} 0 ${225*deg2rad}"/>
+        <xacro:sensor_sick_s300 name="back_right_laser" parent="${prefix}base_link">
+            <origin xyz="-0.606321 -0.345821 0.3095" rpy="${180*deg2rad} 0 ${225*deg2rad}"/>
         </xacro:sensor_sick_s300>
+        <joint name="merged_base_laser_joint" type="fixed"> <!-- front and back laser will be merged into this link -->
+            <origin xyz="0 0 0.234" rpy="0 0 0" />
+            <parent link="${prefix}base_link"/>
+            <child link="${prefix}merged_base_laser_link" />
+        </joint>
+        <link name="merged_base_laser_link" />
    </xacro:macro>
 </robot>

File: vulcano_base_description/urdf/wheels/motor_wheel.urdf.xacro (robot description, xacro)
@@ -3,18 +3,18 @@
   <xacro:property name="M_PI" value="3.1415926535897931" />
   <!-- Wheels -->
-  <xacro:property name="wheel_radius" value="0.093" />
-  <xacro:property name="wheel_height" value="0.14" />
-  <xacro:property name="wheel_mass" value="5.0" /> <!-- in kg-->
-  <xacro:property name="steer_joint_damping" value="2000.0" />
-  <xacro:property name="steer_joint_friction" value="1000.0" />
+  <property name="wheel_radius" value="0.093" />
+  <property name="wheel_height" value="0.14" />
+  <property name="wheel_mass" value="5.0" /> <!-- in kg-->
+  <xacro:property name="steer_joint_damping" value="2.0" />
+  <xacro:property name="steer_joint_friction" value="1.0" />
   <xacro:property name="steer_joint_effort_limit" value="100.0" />
   <xacro:property name="steer_joint_velocity_limit" value="2" />
   <xacro:property name="steer_joint_position_limit" value="2.9" />
-  <xacro:property name="steer_mechanical_reduction" value="1.0" />
-  <xacro:property name="traction_joint_damping" value="1000.0" />
-  <xacro:property name="traction_joint_friction" value="1000.0" />
-  <xacro:property name="traction_joint_effort_limit" value="1000.0" />
-  <xacro:property name="traction_joint_velocity_limit" value="6.28" />
-  <xacro:property name="traction_mechanical_reduction" value="1.0" />
+  <xacro:property name="motor_wheel_mechanical_reduction" value="1.0" />
+  <xacro:property name="wheel_joint_damping" value="0.001" />
+  <xacro:property name="wheel_joint_friction" value="0.001" />
+  <xacro:property name="wheel_joint_effort_limit" value="1000.0" />
+  <xacro:property name="wheel_joint_velocity_limit" value="2000.0" />
+  <xacro:property name="wheel_mechanical_reduction" value="1.0" />
   <xacro:macro name="cylinder_inertia" params="m r h">
     <inertia  ixx="${m*(3*r*r+h*h)/12}" ixy = "0" ixz = "0"
@@ -22,25 +22,26 @@
               izz="${m*r*r/2}" />
   </xacro:macro>
-  <xacro:macro name="motor_wheel" params="prefix parent *origin hq">
+  <xacro:macro name="motor_wheel" params="prefix parent *origin reflect hq">
+  <!-- TODO: check reflect parameter -->
   <!--MOTOR WHEEL -->
-    <joint name="${prefix}wheel_steer_joint" type="revolute">
+    <joint name="${prefix}motor_wheel_joint" type="revolute">
       <parent link="${parent}"/>
-      <child link="${prefix}wheel_steer_link"/>
-      <xacro:insert_block name="origin" />
+      <child link="${prefix}motor_wheel"/>
+      <insert_block name="origin" />
       <axis xyz="0 0 1" rpy="0 0 0" />
       <limit effort="${steer_joint_effort_limit}" velocity="${steer_joint_velocity_limit}" lower="-${steer_joint_position_limit}" upper="${steer_joint_position_limit}"/>
-      <dynamics damping="${steer_joint_damping}" friction="${steer_joint_friction}"/>
+      <joint_properties damping="${steer_joint_damping}" friction="${steer_joint_friction}"/>
     </joint>
-  <transmission name="${prefix}wheel_steer_trans">
+  <transmission name="${prefix}motor_wheel_trans">
      <type>transmission_interface/SimpleTransmission</type>
-     <joint name="${prefix}wheel_steer_joint">
+     <joint name="${prefix}motor_wheel_joint">
         <hardwareInterface>PositionJointInterface</hardwareInterface>
      </joint>
-     <actuator name="${prefix}wheel_steer_motor">
+     <actuator name="${prefix}motor_wheel_motor">
         <hardwareInterface>PositionActuatorInterface</hardwareInterface>
-        <mechanicalReduction>${steer_mechanical_reduction}</mechanicalReduction>
+        <mechanicalReduction>${motor_wheel_mechanical_reduction}</mechanicalReduction>
      </actuator>
   </transmission>
-  <link name="${prefix}wheel_steer_link">
+  <link name="${prefix}motor_wheel">
       <visual>
         <!-- HIGH RESOLUTION WHEELS -->
@@ -48,5 +49,10 @@
           <origin xyz="0 0 0" rpy="0 0 0" />
           <geometry>
-                <mesh filename="package://vulcano_base_description/meshes/wheels/hub.stl" />
+                <xacro:if value="${reflect}">
+                    <mesh filename="package://vulcano_base_description/meshes/wheels/motorwheel_2.dae" />
+                </xacro:if>
+                <xacro:unless value="${reflect}">
+                    <mesh filename="package://vulcano_base_description/meshes/wheels/motorwheel_2.dae" />
+                </xacro:unless>
           </geometry>
         </xacro:if>
@@ -55,5 +61,10 @@
           <origin xyz="0 0 0" rpy="0 0 0" />
           <geometry>
-                <mesh filename="package://vulcano_base_description/meshes/wheels/hub.stl" />
+                <xacro:if value="${reflect}">
+                    <mesh filename="package://vulcano_base_description/meshes/wheels/motorwheel_2.stl" />
+                </xacro:if>
+                <xacro:unless value="${reflect}">
+                    <mesh filename="package://vulcano_base_description/meshes/wheels/motorwheel_2.stl" />
+                </xacro:unless>
           </geometry>
         </xacro:unless>
@@ -62,33 +73,38 @@
         <origin xyz="0 0 0" rpy="0 0 0" />
         <geometry>
-             <mesh filename="package://vulcano_base_description/meshes/wheels/hub.stl" />
+                <xacro:if value="${reflect}">
+                    <mesh filename="package://vulcano_base_description/meshes/wheels/motorwheel_2.dae" />
+                </xacro:if>
+                <xacro:unless value="${reflect}">
+                    <mesh filename="package://vulcano_base_description/meshes/wheels/motorwheel_2.dae" />
+                </xacro:unless>
         </geometry>
       </collision>
       <inertial>
-        <mass value="${wheel_mass}" />
+        <mass value="10" />
         <origin xyz="0 0 0" />
-        <cylinder_inertia  m="${wheel_mass}" r="${wheel_height}" h="${wheel_radius}" /> <!-- TODO: check inertia -->
+        <inertia  ixx="0.01" ixy="0.0"  ixz="0.0"  iyy="0.01"  iyz="0.0"  izz="0.01" />
       </inertial>
     </link>
    <!--WHEEL TIRE -->
-   <joint name="${prefix}wheel_traction_joint" type="continuous">
-        <parent link="${prefix}wheel_steer_link"/>
-        <child link="${prefix}wheel_traction_link"/>
-        <origin xyz="0 0.0035 0" rpy="0 0 ${M_PI}" />
+   <joint name="${prefix}wheel_joint" type="continuous">
+        <parent link="${prefix}motor_wheel"/>
+        <child link="${prefix}wheel"/>
+        <origin xyz="0 0 0" rpy="0 0 ${M_PI}" />
         <axis xyz="0 1 0" rpy="0 0 0" />
-        <limit effort="${traction_joint_effort_limit}" velocity="${traction_joint_velocity_limit}"/>
-        <dynamics damping="${traction_joint_damping}" friction="${traction_joint_friction}"/>
+        <limit effort="${wheel_joint_effort_limit}" velocity="${wheel_joint_velocity_limit}"/>
+        <joint_properties damping="${wheel_joint_damping}" friction="{wheel_joint_friction}"/>
     </joint>
-    <transmission name="${prefix}wheel_traction">
+    <transmission name="${prefix}wheel_trans">
      <type>transmission_interface/SimpleTransmission</type>
-     <joint name="${prefix}wheel_traction_joint">
+     <joint name="${prefix}wheel_joint">
         <hardwareInterface>VelocityJointInterface</hardwareInterface>
      </joint>
-     <actuator name="${prefix}wheel_traction_motor">
+     <actuator name="${prefix}wheel_motor">
        <hardwareInterface>VelocityActuatorInterface</hardwareInterface>
-       <mechanicalReduction>${traction_mechanical_reduction}</mechanicalReduction>
+       <mechanicalReduction>${wheel_mechanical_reduction}</mechanicalReduction>
      </actuator>
     </transmission>
-  <link name="${prefix}wheel_traction_link">
+  <link name="${prefix}wheel">
       <visual>
         <!-- HIGH RESOLUTION WHEELS -->
@@ -96,19 +112,31 @@
           <origin xyz="0 0 0" rpy="0 0 0" />
           <geometry>
-              <mesh filename="package://vulcano_base_description/meshes/wheels/rubber_band.stl" />
+                <xacro:if value="${reflect}">
+                    <mesh filename="package://vulcano_base_description/meshes/wheels/wheel_1.dae" />
+                </xacro:if>
+                <xacro:unless value="${reflect}">
+                    <mesh filename="package://vulcano_base_description/meshes/wheels/wheel_1.dae" />
+                </xacro:unless>
           </geometry>
         </xacro:if>
        <!-- LOW RESOLUTION WHEELS -->
         <xacro:unless value="${hq}">
-          <origin xyz="0 0 0" rpy="0 0 0" />
+          <origin xyz="0 0 0" rpy="${M_PI/2} 0 0" />
           <geometry>
-              <mesh filename="package://vulcano_base_description/meshes/wheels/rubber_band.stl" />
+            <cylinder length="${wheel_height}" radius="${wheel_radius}" />
           </geometry>
         </xacro:unless>
       </visual>
       <collision>
-        <origin xyz="0 0 0" rpy="0 0 0" />
+        <origin xyz="0 0 0" rpy="${M_PI/2} 0 0" />
         <geometry>
-          <mesh filename="package://vulcano_base_description/meshes/wheels/rubber_band.stl" />
+          <!--<xacro:if value="${reflect}">-->
+              <!--<mesh filename="package://vulcano_base_description/meshes/wheels/wheel_1.dae" />-->
+          <!--</xacro:if>-->
+          <!--<xacro:unless value="${reflect}">-->
+              <!--<mesh filename="package://vulcano_base_description/meshes/wheels/wheel_1.dae" />-->
+          <!--</xacro:unless>-->
+          <!-- cylinder length="${wheel_height}" radius="${wheel_radius}" / -->
+          <sphere radius="${wheel_radius}" />
         </geometry>
       </collision>
@@ -119,13 +147,5 @@
       </inertial>
    </link>
-   <!--<gazebo reference="${prefix}wheel_tracion_link">-->
-        <!--<mu1 value="1.0"/>-->
-        <!--<mu2 value="1.0"/>-->
-        <!--[><kp value="10000000.0" /><]-->
-        <!--[><kd value="1.0" /><]-->
-        <!--[><fdir1 value="1 0 0"/><]-->
-        <!--[><turnGravityOff>false</turnGravityOff><]-->
-   <!--</gazebo>-->
-   <!-- gazebo reference="${prefix}motor_wheel_link">
+   <!-- gazebo reference="${prefix}wheel">
         <mu1 value="1.0"/>
         <mu2 value="1.0"/>
