Commit message: description: updated models

File: vulcano_base_description/urdf/bases/base.urdf.xacro (robot description, xacro)
@@ -24,7 +24,7 @@
   <link name="${prefix}base_link">
     <inertial>
-      <mass value="25.0" />
-      <origin xyz="0 0 0" />
-      <inertia  ixx="1.0" ixy="0.0"  ixz="0.0"  iyy="1.0"  iyz="0.0"  izz="1.0" />
+      <mass value="184.0" />
+      <origin xyz="-0.004 0 -0.357" />
+      <inertia  ixx="13.113" ixy="0.131"  ixz="-0.010"  iyy="30.242"  iyz="0.0"  izz="41.3630" />
     </inertial>
     <visual>
@@ -53,7 +53,7 @@
   <link name="${prefix}cabinet_link">
     <inertial>
-      <mass value="15.0" />
-      <origin xyz="0 0 0" />
-      <inertia  ixx="0.1" ixy="0.0"  ixz="0.0"  iyy="0.1"  iyz="0.0"  izz="0.1" />
+      <mass value="96.0" />
+      <origin xyz="-0.089 -0.001 0.00417" />
+      <inertia  ixx="10.783" ixy="-0.137"  ixz="-1.976"  iyy="18.311"  iyz="0.042"  izz="19.866" />
     </inertial>
     <visual>

File: vulcano_base_description/urdf/vulcano_base.urdf.xacro (robot description, xacro)
@@ -42,5 +42,5 @@
         <!-- SENSORS see robotnik_sensors for the specific configuration -->
         <xacro:sensor_imu name="imu" parent="${prefix}base_link">
-          <origin xyz="-0.18 0.0 0.170" rpy="0 0 0"/>
+          <origin xyz="-0.40 0.06 0.75" rpy="0 0 0"/>
         </xacro:sensor_imu>
         <xacro:sensor_sick_s300 name="front_left_laser" parent="${prefix}base_link">

File: vulcano_base_description/urdf/wheels/motor_wheel.urdf.xacro (robot description, xacro)
@@ -10,8 +10,8 @@
   <xacro:property name="steer_joint_effort_limit" value="100.0" />
   <xacro:property name="steer_joint_velocity_limit" value="2" />
-  <xacro:property name="steer_joint_position_limit" value="2.8" />
+  <xacro:property name="steer_joint_position_limit" value="2.9" />
   <xacro:property name="motor_wheel_mechanical_reduction" value="1.0" />
-  <xacro:property name="wheel_joint_damping" value="0.1" />
-  <xacro:property name="wheel_joint_friction" value="0.1" />
+  <xacro:property name="wheel_joint_damping" value="0.001" />
+  <xacro:property name="wheel_joint_friction" value="0.001" />
   <xacro:property name="wheel_joint_effort_limit" value="1000.0" />
   <xacro:property name="wheel_joint_velocity_limit" value="2000.0" />

File: vulcano_torso_description/urdf/guidance/guidance.urdf.xacro (robot description, xacro)
@@ -30,7 +30,7 @@
       </collision>
       <inertial>
-        <origin xyz="0 0 0" rpy="0 0 0"/>
-        <mass value="5"/>
-        <inertia ixx="1.0" ixy="0.0" ixz="0.0" iyy="1.0" iyz="0.0" izz="1.0"/>
+        <origin xyz="0 0 -0.152" rpy="0 0 0"/>
+        <mass value="31"/>
+        <inertia ixx="0.404" ixy="0.0" ixz="0.006" iyy="0.403" iyz="0.0" izz="0.34"/>
       </inertial>
     </link>
@@ -69,7 +69,7 @@
       </collision>
       <inertial>
-        <origin xyz="0 0 0" rpy="0 0 0"/>
-        <mass value="5"/>
-        <inertia ixx="1.0" ixy="0.0" ixz="0.0" iyy="1.0" iyz="0.0" izz="1.0"/>
+        <origin xyz="0.011 -0.001 0.623" rpy="0 0 0"/>
+        <mass value="128"/>
+        <inertia ixx="29.075" ixy="0.013" ixz="0.582" iyy="28.51" iyz="0.009" izz="1.37"/>
       </inertial>
     </link>
@@ -108,7 +108,7 @@
       </collision>
       <inertial>
-        <origin xyz="0 0 0" rpy="0 0 0"/>
-        <mass value="1"/>
-        <inertia ixx="1.0" ixy="0.0" ixz="0.0" iyy="1.0" iyz="0.0" izz="1.0"/>
+        <origin xyz="0.05 0.001 0.432" rpy="0 0 0"/>
+        <mass value="41"/>
+        <inertia ixx="1.881" ixy="-0.004" ixz="0.084" iyy="1.122" iyz="-0.008" izz="1.295"/>
       </inertial>
     </link>

Commit message: description: updated model to new version

File: vulcano_base_description/urdf/bases/base.urdf.xacro (robot description, xacro)
@@ -15,5 +15,5 @@
       </visual>
     </link>
-    <joint name="base_footprint_joint" type="fixed">
+    <joint name="${prefix}base_footprint_joint" type="fixed">
       <origin xyz="0 0 ${wheel_radius}" rpy="0 0 0" /> <!-- ${wheel_radius} property must be defined inside wheel description -->
       <parent link="${prefix}base_footprint"/>
@@ -23,21 +23,16 @@
   <!-- BASE_LINK -->
   <link name="${prefix}base_link">
-    <inertial>
-      <mass value="184.0" />
-      <origin xyz="-0.004 0 -0.357" />
-      <inertia  ixx="13.113" ixy="0.131"  ixz="-0.010"  iyy="30.242"  iyz="0.0"  izz="41.3630" />
-    </inertial>
+    <!--<inertial>-->
+      <!--<mass value="184.0" />-->
+      <!--<origin xyz="-0.004 0 -0.357" />-->
+      <!--<inertia  ixx="13.113" ixy="0.131"  ixz="-0.010"  iyy="30.242"  iyz="0.0"  izz="41.3630" />-->
+    <!--</inertial>-->
     <visual>
        <origin xyz="0 0 0" rpy="0 0 0" />
-       <xacro:if value="${hq}">
+       <!--<xacro:if value="${hq}">-->
        <geometry>
-	     <mesh filename="package://vulcano_base_description/meshes/bases/vulcano_base_chassis.dae"/>
+	     <mesh filename="package://vulcano_base_description/meshes/bases/cabinet.stl"/>
        </geometry>
-       </xacro:if>
-       <xacro:unless value="${hq}">
-       <geometry>
-	     <mesh filename="package://vulcano_base_description/meshes/bases/vulcano_base_chassis.dae"/>
-       </geometry>
-       </xacro:unless>
+       <!--</xacro:if>-->
        <material name="darkgrey">
          <color rgba="0.1 0.1 0.1 1"/>
@@ -47,42 +42,8 @@
        <origin xyz="0 0 0" rpy="0 0 0 " />
        <geometry>
-         <mesh filename="package://vulcano_base_description/meshes/bases/vulcano_base_chassis.dae"/>
+	     <mesh filename="package://vulcano_base_description/meshes/bases/cabinet.stl"/>
        </geometry>
     </collision>
   </link>
-  <link name="${prefix}cabinet_link">
-    <inertial>
-      <mass value="96.0" />
-      <origin xyz="-0.089 -0.001 0.00417" />
-      <inertia  ixx="10.783" ixy="-0.137"  ixz="-1.976"  iyy="18.311"  iyz="0.042"  izz="19.866" />
-    </inertial>
-    <visual>
-       <origin xyz="0 0 0" rpy="0 0 0" />
-       <xacro:if value="${hq}">
-       <geometry>
-	     <mesh filename="package://vulcano_base_description/meshes/bases/vulcano_base_cabinet.dae"/>
-       </geometry>
-       </xacro:if>
-       <xacro:unless value="${hq}">
-       <geometry>
-	     <mesh filename="package://vulcano_base_description/meshes/bases/vulcano_base_cabinet.dae"/>
-       </geometry>
-       </xacro:unless>
-       <material name="darkgrey">
-         <color rgba="0.1 0.1 0.1 1"/>
-       </material>
-    </visual>
-    <collision>
-       <origin xyz="0 0 0" rpy="0 0 0 " />
-       <geometry>
-         <mesh filename="package://vulcano_base_description/meshes/bases/vulcano_base_cabinet.dae"/>
-       </geometry>
-    </collision>
-  </link>
-  <joint name="${prefix}cabinet_joint" type="fixed">
-    <origin xyz="0 0 0.234" rpy="0 0 0" />
-    <parent link="${prefix}base_link"/>
-    <child link="${prefix}cabinet_link" />
-  </joint>
   </xacro:macro>
 </robot>

File: vulcano_base_description/urdf/wheels/motor_wheel.urdf.xacro (robot description, xacro)
@@ -3,7 +3,7 @@
   <xacro:property name="M_PI" value="3.1415926535897931" />
   <!-- Wheels -->
-  <property name="wheel_radius" value="0.093" />
-  <property name="wheel_height" value="0.14" />
-  <property name="wheel_mass" value="5.0" /> <!-- in kg-->
+  <xacro:property name="wheel_radius" value="0.093" />
+  <xacro:property name="wheel_height" value="0.14" />
+  <xacro:property name="wheel_mass" value="5.0" /> <!-- in kg-->
   <xacro:property name="steer_joint_damping" value="2.0" />
   <xacro:property name="steer_joint_friction" value="1.0" />
@@ -28,5 +28,5 @@
       <parent link="${parent}"/>
       <child link="${prefix}wheel_steer_link"/>
-      <insert_block name="origin" />
+      <xacro:insert_block name="origin" />
       <axis xyz="0 0 1" rpy="0 0 0" />
       <limit effort="${steer_joint_effort_limit}" velocity="${steer_joint_velocity_limit}" lower="-${steer_joint_position_limit}" upper="${steer_joint_position_limit}"/>
@@ -50,8 +50,8 @@
           <geometry>
                 <xacro:if value="${reflect}">
-                    <mesh filename="package://vulcano_base_description/meshes/wheels/motorwheel_2.dae" />
+                    <mesh filename="package://vulcano_base_description/meshes/wheels/hub.stl" />
                 </xacro:if>
                 <xacro:unless value="${reflect}">
-                    <mesh filename="package://vulcano_base_description/meshes/wheels/motorwheel_2.dae" />
+                    <mesh filename="package://vulcano_base_description/meshes/wheels/hub.stl" />
                 </xacro:unless>
           </geometry>
@@ -62,8 +62,8 @@
           <geometry>
                 <xacro:if value="${reflect}">
-                    <mesh filename="package://vulcano_base_description/meshes/wheels/motorwheel_2.stl" />
+                    <mesh filename="package://vulcano_base_description/meshes/wheels/hub.stl" />
                 </xacro:if>
                 <xacro:unless value="${reflect}">
-                    <mesh filename="package://vulcano_base_description/meshes/wheels/motorwheel_2.stl" />
+                    <mesh filename="package://vulcano_base_description/meshes/wheels/hub.stl" />
                 </xacro:unless>
           </geometry>
@@ -74,8 +74,8 @@
         <geometry>
                 <xacro:if value="${reflect}">
-                    <mesh filename="package://vulcano_base_description/meshes/wheels/motorwheel_2.dae" />
+                    <mesh filename="package://vulcano_base_description/meshes/wheels/hub.stl" />
                 </xacro:if>
                 <xacro:unless value="${reflect}">
-                    <mesh filename="package://vulcano_base_description/meshes/wheels/motorwheel_2.dae" />
+                    <mesh filename="package://vulcano_base_description/meshes/wheels/hub.stl" />
                 </xacro:unless>
         </geometry>
@@ -91,5 +91,5 @@
         <parent link="${prefix}wheel_steer_link"/>
         <child link="${prefix}wheel_traction_link"/>
-        <origin xyz="0 0 0" rpy="0 0 ${M_PI}" />
+        <origin xyz="0 0.0035 0" rpy="0 0 ${M_PI}" />
         <axis xyz="0 1 0" rpy="0 0 0" />
         <limit effort="${traction_joint_effort_limit}" velocity="${traction_joint_velocity_limit}"/>
@@ -113,8 +113,8 @@
           <geometry>
                 <xacro:if value="${reflect}">
-                    <mesh filename="package://vulcano_base_description/meshes/wheels/wheel_1.dae" />
+                    <mesh filename="package://vulcano_base_description/meshes/wheels/rubber_band.stl" />
                 </xacro:if>
                 <xacro:unless value="${reflect}">
-                    <mesh filename="package://vulcano_base_description/meshes/wheels/wheel_1.dae" />
+                    <mesh filename="package://vulcano_base_description/meshes/wheels/rubber_band.stl" />
                 </xacro:unless>
           </geometry>
@@ -138,5 +138,6 @@
           <!--</xacro:unless>-->
           <!-- cylinder length="${wheel_height}" radius="${wheel_radius}" / -->
-          <sphere radius="${wheel_radius}" />
+          <!--sphere radius="${wheel_radius}" /-->
+          <mesh filename="package://vulcano_base_description/meshes/wheels/rubber_band.stl" />
         </geometry>
       </collision>

File: vulcano_description/robots/vulcano_robot.urdf.xacro (robot description, xacro)
@@ -20,5 +20,5 @@
   <!-- Fix torso to base -->
   <joint name="base_torso_joint" type="fixed">
-    <origin xyz="0.47 0.0 0.474" rpy="0.0 0.0 0.0"/>
+    <origin xyz="0.5607 0.0 0.4845" rpy="0.0 0.0 0.0"/>
     <parent link="base_link"/>
     <child link="torso_base_link"/>
@@ -28,6 +28,6 @@
   <!-- Fix right arm to torso -->
   <joint name="torso_right_arm_base_joint" type="fixed">
-    <origin xyz="-0.1622 0.275533 0.021967" rpy="0 ${-PI/4.0} ${-PI/2.0}"/>  <!-- TODO: set correct orientation -->
-    <parent link="torso_tkd668_link"/>
+    <origin xyz="0.16870 0.28753 -0.12303" rpy="0 ${-PI/4.0} ${-PI/2.0}"/>
+    <parent link="torso_guidance_elevation_link"/>
     <child link="right_arm_base_link"/>
   </joint>
@@ -35,6 +35,6 @@
   <!-- Fix left arm to torso -->
   <joint name="torso_left_arm_base_joint" type="fixed">
-    <origin xyz="-0.1622 -0.275533 0.021967" rpy="0 ${PI/4.0} ${-PI/2.0}"/>
-    <parent link="torso_tkd668_link"/>
+    <origin xyz="0.16870 -0.28753 -0.12303" rpy="0 ${PI/4.0} ${-PI/2.0}"/>
+    <parent link="torso_guidance_elevation_link"/>
     <child link="left_arm_base_link"/>
   </joint>

File: vulcano_torso_description/urdf/guidance/guidance.urdf.xacro (robot description, xacro)
@@ -13,26 +13,5 @@
       <axis xyz="0 0 1"/>
     </joint>
-    <link name="${prefix}torso_guidance_base_link">
-      <visual>
-        <origin xyz="0 0 0" rpy="0 0 0"/>
-        <geometry>
-          <mesh filename="package://vulcano_torso_description/meshes/guidance/base.stl"/>
-        </geometry>
-       <material name="darkgrey">
-         <color rgba="0.1 0.1 0.1 1"/>
-       </material>
-      </visual>
-      <collision>
-        <origin xyz="0 0 0" rpy="0 0 0"/>
-        <geometry>
-          <mesh filename="package://vulcano_torso_description/meshes/guidance/base.stl"/>
-        </geometry>
-      </collision>
-      <inertial>
-        <origin xyz="0 0 -0.152" rpy="0 0 0"/>
-        <mass value="31"/>
-        <inertia ixx="0.404" ixy="0.0" ixz="0.006" iyy="0.403" iyz="0.0" izz="0.34"/>
-      </inertial>
-    </link>
+    <link name="${prefix}torso_guidance_base_link"/>
     <joint name="${prefix}torso_guidance_revolution_joint" type="revolute">
       <origin xyz="0 0 0" rpy="0 0 ${PI}"/>
@@ -56,5 +35,5 @@
         <origin xyz="0 0 0" rpy="0 0 0"/>
         <geometry>
-          <mesh filename="package://vulcano_torso_description/meshes/guidance/main.stl"/>
+          <mesh filename="package://vulcano_torso_description/meshes/guidance/guidance.stl"/>
         </geometry>
        <material name="darkgrey">
@@ -65,5 +44,5 @@
         <origin xyz="0 0 0" rpy="0 0 0"/>
         <geometry>
-          <mesh filename="package://vulcano_torso_description/meshes/guidance/main.stl"/>
+          <mesh filename="package://vulcano_torso_description/meshes/guidance/guidance.stl"/>
         </geometry>
       </collision>
@@ -75,9 +54,9 @@
     </link>
     <joint name="${prefix}torso_guidance_elevation_joint" type="prismatic">
-      <origin xyz="0 0 0.115" rpy="0 0 0"/>
+      <origin xyz="-0.1687 0 0.720" rpy="0 0 0"/>
       <parent link="${prefix}torso_guidance_revolution_link"/>
       <child link="${prefix}torso_guidance_elevation_link"/>
       <axis xyz="0 0 1"/>
-      <limit lower="0.0" upper="0.68" effort="100" velocity="0.08"/>
+      <limit lower="0.0" upper="0.6" effort="100" velocity="0.08"/>
       <dynamics friction="100000" damping="10000"/>
     </joint>
@@ -113,27 +92,4 @@
       </inertial>
     </link>
-    <joint name="${prefix}torso_tkd668_joint" type="fixed">
-      <origin xyz="0.164 0 0.449" rpy="0 0 0"/>
-      <parent link="${prefix}torso_guidance_elevation_link"/>
-      <child link="${prefix}torso_tkd668_link"/>
-      <axis xyz="0 0 1"/>
-    </joint>
-    <link name="${prefix}torso_tkd668_link">
-      <visual>
-        <origin xyz="0 0 0" rpy="0 0 0"/>
-        <geometry>
-          <mesh filename="package://vulcano_torso_description/meshes/guidance/tkd668.stl"/>
-        </geometry>
-       <material name="darkgrey">
-         <color rgba="0.1 0.1 0.1 1"/>
-       </material>
-      </visual>
-      <collision>
-        <origin xyz="0 0 0" rpy="0 0 0"/>
-        <geometry>
-          <mesh filename="package://vulcano_torso_description/meshes/guidance/tkd668.stl"/>
-        </geometry>
-      </collision>
-    </link>
   </xacro:macro>
 </robot>

File: vulcano_torso_description/urdf/tube_support/tube_support.urdf.xacro (robot description, xacro)
@@ -4,5 +4,5 @@
   <xacro:macro name="tube_support" params="prefix parent *origin *box">
     <joint name="${prefix}tube_support_joint" type="fixed">
-        <insert_block name="origin" />
+        <xacro:insert_block name="origin" />
         <parent link="${parent}" />
         <child link="${prefix}tube_support_link"/>
@@ -12,5 +12,5 @@
         <origin xyz="0 0 0" rpy="0 0 0" />
         <geometry>
-            <insert_block name="box" />
+            <xacro:insert_block name="box" />
         </geometry>
       </collision>
