Commit message: updated models to match new names

File: vulcano_base_description/urdf/bases/base.urdf.xacro (robot description, xacro)
@@ -5,4 +5,9 @@
   <xacro:property name="PI" value="3.1415926535897931"/>
   <xacro:property name="wheel_width" value="0.075" />
+  <xacro:macro name="box_inertia" params="m x y z">
+    <inertia  ixx="${m*(y*y+z*z)/12}" ixy = "0" ixz = "0"
+              iyy="${m*(x*x+z*z)/12}" iyz = "0"
+              izz="${m*(x*x+y*y)/12}" />
+  </xacro:macro>
   <!-- BASE FOOTPRINT -->
   <xacro:if value="${publish_bf}">
@@ -15,5 +20,5 @@
       </visual>
     </link>
-    <joint name="base_footprint_joint" type="fixed">
+    <joint name="${prefix}base_footprint_joint" type="fixed">
       <origin xyz="0 0 ${wheel_radius}" rpy="0 0 0" /> <!-- ${wheel_radius} property must be defined inside wheel description -->
       <parent link="${prefix}base_footprint"/>

File: vulcano_base_description/urdf/vulcano_base.urdf.xacro (robot description, xacro)
@@ -41,19 +41,19 @@
         </xacro:motor_wheel>
         <!-- SENSORS see robotnik_sensors for the specific configuration -->
-        <xacro:sensor_imu name="imu" parent="${prefix}base_link">
+        <xacro:sensor_imu prefix="${prefix}imu" parent="${prefix}base_link">
           <origin xyz="-0.40 0.06 0.75" rpy="0 0 0"/>
         </xacro:sensor_imu>
-        <xacro:sensor_sick_s300 name="front_left_laser" parent="${prefix}base_link">
+        <xacro:sensor_sick_s300 prefix="${prefix}front_left_laser" parent="${prefix}base_link">
             <origin xyz="0.606321 0.345821 0.3095" rpy="${180*deg2rad} 0 ${45*deg2rad}"/>
         </xacro:sensor_sick_s300>
-        <xacro:sensor_sick_s300 name="back_right_laser" parent="${prefix}base_link">
+        <xacro:sensor_sick_s300 prefix="${prefix}back_right_laser" parent="${prefix}base_link">
             <origin xyz="-0.606321 -0.345821 0.3095" rpy="${180*deg2rad} 0 ${225*deg2rad}"/>
         </xacro:sensor_sick_s300>
-        <joint name="merged_base_laser_joint" type="fixed"> <!-- front and back laser will be merged into this link -->
+        <joint name="${prefix}merged_base_laser_joint" type="fixed"> <!-- front and back laser will be merged into this link -->
             <origin xyz="0 0 0.234" rpy="0 0 0" />
             <parent link="${prefix}base_link"/>
             <child link="${prefix}merged_base_laser_link" />
         </joint>
-        <link name="merged_base_laser_link" />
+        <link name="${prefix}merged_base_laser_link" />
    </xacro:macro>
 </robot>

File: vulcano_base_description/urdf/wheels/motor_wheel.urdf.xacro (robot description, xacro)
@@ -3,18 +3,18 @@
   <xacro:property name="M_PI" value="3.1415926535897931" />
   <!-- Wheels -->
-  <property name="wheel_radius" value="0.093" />
-  <property name="wheel_height" value="0.14" />
-  <property name="wheel_mass" value="5.0" /> <!-- in kg-->
-  <xacro:property name="steer_joint_damping" value="2.0" />
-  <xacro:property name="steer_joint_friction" value="1.0" />
+  <xacro:property name="wheel_radius" value="0.093" />
+  <xacro:property name="wheel_height" value="0.14" />
+  <xacro:property name="wheel_mass" value="5.0" /> <!-- in kg-->
+  <xacro:property name="steer_joint_damping" value="2000.0" />
+  <xacro:property name="steer_joint_friction" value="1000.0" />
   <xacro:property name="steer_joint_effort_limit" value="100.0" />
   <xacro:property name="steer_joint_velocity_limit" value="2" />
   <xacro:property name="steer_joint_position_limit" value="2.9" />
-  <xacro:property name="motor_wheel_mechanical_reduction" value="1.0" />
-  <xacro:property name="wheel_joint_damping" value="0.001" />
-  <xacro:property name="wheel_joint_friction" value="0.001" />
-  <xacro:property name="wheel_joint_effort_limit" value="1000.0" />
-  <xacro:property name="wheel_joint_velocity_limit" value="2000.0" />
-  <xacro:property name="wheel_mechanical_reduction" value="1.0" />
+  <xacro:property name="steer_mechanical_reduction" value="1.0" />
+  <xacro:property name="traction_joint_damping" value="1000.0" />
+  <xacro:property name="traction_joint_friction" value="1000.0" />
+  <xacro:property name="traction_joint_effort_limit" value="1000.0" />
+  <xacro:property name="traction_joint_velocity_limit" value="6.28" />
+  <xacro:property name="traction_mechanical_reduction" value="1.0" />
   <xacro:macro name="cylinder_inertia" params="m r h">
     <inertia  ixx="${m*(3*r*r+h*h)/12}" ixy = "0" ixz = "0"
@@ -25,23 +25,23 @@
   <!-- TODO: check reflect parameter -->
   <!--MOTOR WHEEL -->
-    <joint name="${prefix}motor_wheel_joint" type="revolute">
+    <joint name="${prefix}wheel_steer_joint" type="revolute">
       <parent link="${parent}"/>
-      <child link="${prefix}motor_wheel"/>
-      <insert_block name="origin" />
+      <child link="${prefix}wheel_steer_link"/>
+      <xacro:insert_block name="origin" />
       <axis xyz="0 0 1" rpy="0 0 0" />
       <limit effort="${steer_joint_effort_limit}" velocity="${steer_joint_velocity_limit}" lower="-${steer_joint_position_limit}" upper="${steer_joint_position_limit}"/>
-      <joint_properties damping="${steer_joint_damping}" friction="${steer_joint_friction}"/>
+      <dynamics damping="${steer_joint_damping}" friction="${steer_joint_friction}"/>
     </joint>
-  <transmission name="${prefix}motor_wheel_trans">
+  <transmission name="${prefix}wheel_steer_trans">
      <type>transmission_interface/SimpleTransmission</type>
-     <joint name="${prefix}motor_wheel_joint">
+     <joint name="${prefix}wheel_steer_joint">
         <hardwareInterface>PositionJointInterface</hardwareInterface>
      </joint>
-     <actuator name="${prefix}motor_wheel_motor">
+     <actuator name="${prefix}wheel_steer_motor">
         <hardwareInterface>PositionActuatorInterface</hardwareInterface>
-        <mechanicalReduction>${motor_wheel_mechanical_reduction}</mechanicalReduction>
+        <mechanicalReduction>${steer_mechanical_reduction}</mechanicalReduction>
      </actuator>
   </transmission>
-  <link name="${prefix}motor_wheel">
+  <link name="${prefix}wheel_steer_link">
       <visual>
         <!-- HIGH RESOLUTION WHEELS -->
@@ -82,29 +82,29 @@
       </collision>
       <inertial>
-        <mass value="10" />
+        <mass value="${wheel_mass}" />
         <origin xyz="0 0 0" />
-        <inertia  ixx="0.01" ixy="0.0"  ixz="0.0"  iyy="0.01"  iyz="0.0"  izz="0.01" />
+        <cylinder_inertia  m="${wheel_mass}" r="${wheel_height}" h="${wheel_radius}" /> <!-- TODO: check inertia -->
       </inertial>
     </link>
    <!--WHEEL TIRE -->
-   <joint name="${prefix}wheel_joint" type="continuous">
-        <parent link="${prefix}motor_wheel"/>
-        <child link="${prefix}wheel"/>
+   <joint name="${prefix}wheel_traction_joint" type="continuous">
+        <parent link="${prefix}wheel_steer_link"/>
+        <child link="${prefix}wheel_traction_link"/>
         <origin xyz="0 0 0" rpy="0 0 ${M_PI}" />
         <axis xyz="0 1 0" rpy="0 0 0" />
-        <limit effort="${wheel_joint_effort_limit}" velocity="${wheel_joint_velocity_limit}"/>
-        <joint_properties damping="${wheel_joint_damping}" friction="{wheel_joint_friction}"/>
+        <limit effort="${traction_joint_effort_limit}" velocity="${traction_joint_velocity_limit}"/>
+        <dynamics damping="${traction_joint_damping}" friction="${traction_joint_friction}"/>
     </joint>
-    <transmission name="${prefix}wheel_trans">
+    <transmission name="${prefix}wheel_traction">
      <type>transmission_interface/SimpleTransmission</type>
-     <joint name="${prefix}wheel_joint">
+     <joint name="${prefix}wheel_traction_joint">
         <hardwareInterface>VelocityJointInterface</hardwareInterface>
      </joint>
-     <actuator name="${prefix}wheel_motor">
+     <actuator name="${prefix}wheel_traction_motor">
        <hardwareInterface>VelocityActuatorInterface</hardwareInterface>
-       <mechanicalReduction>${wheel_mechanical_reduction}</mechanicalReduction>
+       <mechanicalReduction>${traction_mechanical_reduction}</mechanicalReduction>
      </actuator>
     </transmission>
-  <link name="${prefix}wheel">
+  <link name="${prefix}wheel_traction_link">
       <visual>
         <!-- HIGH RESOLUTION WHEELS -->
@@ -147,5 +147,13 @@
       </inertial>
    </link>
-   <!-- gazebo reference="${prefix}wheel">
+   <!--<gazebo reference="${prefix}wheel_tracion_link">-->
+        <!--<mu1 value="1.0"/>-->
+        <!--<mu2 value="1.0"/>-->
+        <!--[><kp value="10000000.0" /><]-->
+        <!--[><kd value="1.0" /><]-->
+        <!--[><fdir1 value="1 0 0"/><]-->
+        <!--[><turnGravityOff>false</turnGravityOff><]-->
+   <!--</gazebo>-->
+   <!-- gazebo reference="${prefix}motor_wheel_link">
         <mu1 value="1.0"/>
         <mu2 value="1.0"/>
