Commit message: vulcano_torso_description: added pantilt

File: vulcano_torso_description/urdf/guidance/guidance.urdf.xacro (robot description, xacro)
@@ -6,16 +6,8 @@
   <xacro:property name="z_elevation_joint" value="0.442"/>
   <!-- Define the torso -->
-  <xacro:macro name="torso" params="prefix hq">
-    <link name="${prefix}torso_base_link">
-      <inertial>
-        <origin xyz="0 0 0" rpy="0 0 0 "/>
-        <mass value="5"/> <!-- TODO: check masses -->
-        <inertia ixx="1.0" ixy="0.0" ixz="0.0" iyy="1.0" iyz="0.0" izz="1.0"/>
-      </inertial>
-    </link>
+  <xacro:macro name="guidance" params="prefix parent hq">
     <joint name="${prefix}torso_guidance_base_joint" type="fixed">
-      <!--<origin xyz="0.47 0 0.474" rpy="0 0 0"/>-->
       <origin xyz="0.0 0.0 0.0" rpy="0 0 0"/>
-      <parent link="${prefix}torso_base_link"/>
+      <parent link="${parent}"/>
       <child link="${prefix}torso_guidance_base_link"/>
       <axis xyz="0 0 1"/>
@@ -25,5 +17,5 @@
         <origin xyz="0 0 0" rpy="0 0 0"/>
         <geometry>
-          <mesh filename="package://vulcano_torso_description/meshes/guidance_base.stl"/>
+          <mesh filename="package://vulcano_torso_description/meshes/guidance/base.stl"/>
         </geometry>
        <material name="darkgrey">
@@ -34,5 +26,5 @@
         <origin xyz="0 0 0" rpy="0 0 0"/>
         <geometry>
-          <mesh filename="package://vulcano_torso_description/meshes/guidance_base.stl"/>
+          <mesh filename="package://vulcano_torso_description/meshes/guidance/base.stl"/>
         </geometry>
       </collision>
@@ -57,5 +49,5 @@
       <joint name="${prefix}torso_revolution_joint">
         <!--<hardwareInterface>EffortJointInterface</hardwareInterface>-->
-        <hardwareInterface>PositionJointInterface</hardwareInterface><!-- TODO: PositionJointInterface? EffortJointInterface? -->
+        <hardwareInterface>PositionJointInterface</hardwareInterface> <!-- TODO: PositionJointInterface? EffortJointInterface?  VelocityJointInterface? -->
       </joint>
       <actuator name="${prefix}torso_revolution_motor">
@@ -68,5 +60,5 @@
         <origin xyz="0 0 0" rpy="0 0 0"/>
         <geometry>
-          <mesh filename="package://vulcano_torso_description/meshes/guidance_main.stl"/>
+          <mesh filename="package://vulcano_torso_description/meshes/guidance/main.stl"/>
         </geometry>
        <material name="darkgrey">
@@ -77,5 +69,5 @@
         <origin xyz="0 0 0" rpy="0 0 0"/>
         <geometry>
-          <mesh filename="package://vulcano_torso_description/meshes/guidance_main.stl"/>
+          <mesh filename="package://vulcano_torso_description/meshes/guidance/main.stl"/>
         </geometry>
       </collision>
@@ -98,5 +90,5 @@
       <joint name="${prefix}torso_elevation_joint">
         <!--<hardwareInterface>EffortJointInterface</hardwareInterface>-->
-        <hardwareInterface>PositionJointInterface</hardwareInterface><!-- TODO: PositionJointInterface? EffortJointInterface? -->
+        <hardwareInterface>PositionJointInterface</hardwareInterface> <!-- TODO: PositionJointInterface? EffortJointInterface?  VelocityJointInterface? -->
       </joint>
       <actuator name="${prefix}torso_elevation_motor">
@@ -109,5 +101,5 @@
         <origin xyz="0 0 0" rpy="0 0 0"/>
         <geometry>
-          <mesh filename="package://vulcano_torso_description/meshes/guidance_slide.stl"/>
+          <mesh filename="package://vulcano_torso_description/meshes/guidance/slide.stl"/>
         </geometry>
        <material name="darkgrey">
@@ -118,5 +110,5 @@
         <origin xyz="0 0 0" rpy="0 0 0"/>
         <geometry>
-          <mesh filename="package://vulcano_torso_description/meshes/guidance_slide.stl"/>
+          <mesh filename="package://vulcano_torso_description/meshes/guidance/slide.stl"/>
         </geometry>
       </collision>
@@ -137,5 +129,5 @@
         <origin xyz="0 0 0" rpy="0 0 0"/>
         <geometry>
-          <mesh filename="package://vulcano_torso_description/meshes/tkd668.stl"/>
+          <mesh filename="package://vulcano_torso_description/meshes/guidance/tkd668.stl"/>
         </geometry>
        <material name="darkgrey">
@@ -146,5 +138,5 @@
         <origin xyz="0 0 0" rpy="0 0 0"/>
         <geometry>
-          <mesh filename="package://vulcano_torso_description/meshes/tkd668.stl"/>
+          <mesh filename="package://vulcano_torso_description/meshes/guidance/tkd668.stl"/>
         </geometry>
       </collision>

File: vulcano_torso_description/urdf/vulcano_torso.urdf.xacro (robot description, xacro)
@@ -4,10 +4,43 @@
     <!-- Imported elements -->
     <!-- ***************** -->
+    <xacro:property name="deg2rad" value="0.01745329251"/>
     <!-- First we import all posible elements defined in the urdf.xacro files. All these elements are defined as macro:xacros -->
     <!-- Include vulcano torso elements -->
-    <xacro:include filename="$(find vulcano_torso_description)/urdf/torso/torso.urdf.xacro"/>
+    <xacro:include filename="$(find vulcano_torso_description)/urdf/guidance/guidance.urdf.xacro"/>
+    <xacro:include filename="$(find vulcano_torso_description)/urdf/pantilt/pantilt.urdf.xacro"/>
     <xacro:include filename="$(find robotnik_sensors)/urdf/all_sensors.urdf.xacro" />
-    <xacro:macro name="vulcano_torso" params="prefix hq">
-        <xacro:torso prefix="${prefix}" hq="${hq}"/>
+    <xacro:macro name="vulcano_torso" params="prefix hq"> <!-- TODO: check hq variable -->
+        <link name="${prefix}torso_base_link">
+            <inertial>
+                <origin xyz="0 0 0" rpy="0 0 0 "/>
+                <mass value="5"/> <!-- TODO: check masses -->
+            <inertia ixx="1.0" ixy="0.0" ixz="0.0" iyy="1.0" iyz="0.0" izz="1.0"/>
+            </inertial>
+        </link>
+        <xacro:guidance prefix="${prefix}" parent="${prefix}torso_base_link" hq="${hq}"/>
+        <joint name="${prefix}torso_guidance_pantilt_joint" type="fixed">
+          <origin xyz="-0.191 0.0 1.178" rpy="0 0 ${180*deg2rad}"/>
+          <parent link="${prefix}torso_guidance_main_link"/>
+          <child link="${prefix}torso_guidance_pantilt_link"/>
+          <axis xyz="0 0 1"/>
+        </joint>
+        <link name="${prefix}torso_guidance_pantilt_link">
+            <inertial>
+                <origin xyz="0 0 0" rpy="0 0 0 "/>
+                <mass value="5"/> <!-- TODO: check masses -->
+            <inertia ixx="1.0" ixy="0.0" ixz="0.0" iyy="1.0" iyz="0.0" izz="1.0"/>
+            </inertial>
+        </link>
+        <xacro:pantilt prefix="${prefix}" parent="${prefix}torso_guidance_pantilt_link" hq="${hq}"/>
+        <!-- TODO: check kinect2 position -->
+        <xacro:sensor_kinectv2 name="${prefix}torso_kinect" parent="${prefix}torso_pantilt_link" base="true">
+            <origin xyz="0.01255 0 0.066" rpy="0 0 0"/>
+        </xacro:sensor_kinectv2>
+        <xacro:sensor_ueye_cp_gige name="${prefix}torso_ueye_left" parent="${prefix}torso_pantilt_link">
+            <origin xyz="0.0258 -0.14975 0.0165" rpy="0 0 0"/>
+        </xacro:sensor_ueye_cp_gige>
+        <xacro:sensor_ueye_cp_gige name="${prefix}torso_ueye_right" parent="${prefix}torso_pantilt_link">
+            <origin xyz="0.0258 0.14975 0.0165" rpy="0 0 0"/>
+        </xacro:sensor_ueye_cp_gige>
     </xacro:macro>
 </robot>

Commit message: vulcano_torso_description: updated guidance model

File: vulcano_torso_description/urdf/guidance/guidance.urdf.xacro (robot description, xacro)
@@ -37,10 +37,9 @@
     <joint name="${prefix}torso_revolution_joint" type="revolute">
       <!-- TODO: especificar zona muerta, limites de articulacion y parametros de simulacion -->
-      <!--origin xyz="0 0 0" rpy="0 0 ${60*deg2rad}" /-->
       <origin xyz="0 0 0" rpy="0 0 ${PI}"/>
       <parent link="${prefix}torso_guidance_base_link"/>
       <child link="${prefix}torso_guidance_main_link"/>
       <axis xyz="0 0 1"/>
-      <limit lower="${-172*deg2rad}" upper="${172*deg2rad}" effort="100" velocity="100"/>
+      <limit lower="${-135*deg2rad}" upper="${225*deg2rad}" effort="100" velocity="100"/>
       <dynamics friction="1000" damping="1000"/>
     </joint>

Commit message: vulcano_torso_description: update link and joints names

File: vulcano_torso_description/urdf/guidance/guidance.urdf.xacro (robot description, xacro)
@@ -35,25 +35,25 @@
       </inertial>
     </link>
-    <joint name="${prefix}torso_revolution_joint" type="revolute">
+    <joint name="${prefix}torso_guidance_revolution_joint" type="revolute">
       <!-- TODO: especificar zona muerta, limites de articulacion y parametros de simulacion -->
       <origin xyz="0 0 0" rpy="0 0 ${PI}"/>
       <parent link="${prefix}torso_guidance_base_link"/>
-      <child link="${prefix}torso_guidance_main_link"/>
+      <child link="${prefix}torso_guidance_revolution_link"/>
       <axis xyz="0 0 1"/>
       <limit lower="${-135*deg2rad}" upper="${225*deg2rad}" effort="100" velocity="100"/>
       <dynamics friction="1000" damping="1000"/>
     </joint>
-	<transmission name="${prefix}torso_revolution_trans">
+	<transmission name="${prefix}torso_guidance_revolution_trans">
       <type>transmission_interface/SimpleTransmission</type>
-      <joint name="${prefix}torso_revolution_joint">
+      <joint name="${prefix}torso_guidance_revolution_joint">
         <!--<hardwareInterface>EffortJointInterface</hardwareInterface>-->
         <hardwareInterface>PositionJointInterface</hardwareInterface> <!-- TODO: PositionJointInterface? EffortJointInterface?  VelocityJointInterface? -->
       </joint>
-      <actuator name="${prefix}torso_revolution_motor">
+      <actuator name="${prefix}torso_guidance_revolution_motor">
         <mechanicalReduction>1</mechanicalReduction>
         <hardwareInterface>EffortJointInterface</hardwareInterface>
       </actuator>
     </transmission>
-    <link name="${prefix}torso_guidance_main_link">
+    <link name="${prefix}torso_guidance_revolution_link">
       <visual>
         <origin xyz="0 0 0" rpy="0 0 0"/>
@@ -77,24 +77,24 @@
       </inertial>
     </link>
-    <joint name="${prefix}torso_elevation_joint" type="prismatic">
+    <joint name="${prefix}torso_guidance_elevation_joint" type="prismatic">
       <!-- TODO: especificar limites de articulacion y parametros de simulacion -->
       <origin xyz="0 0 0.115" rpy="0 0 0"/>
-      <parent link="${prefix}torso_guidance_main_link"/>
-      <child link="${prefix}torso_guidance_slide_link"/>
+      <parent link="${prefix}torso_guidance_revolution_link"/>
+      <child link="${prefix}torso_guidance_elevation_link"/>
       <axis xyz="0 0 1"/>
       <limit lower="0" upper="0.739" effort="100" velocity="100"/>
     </joint>
-	<transmission name="${prefix}torso_elevation_trans">
+	<transmission name="${prefix}torso_guidance_elevation_trans">
       <type>transmission_interface/SimpleTransmission</type>
-      <joint name="${prefix}torso_elevation_joint">
+      <joint name="${prefix}torso_guidance_elevation_joint">
         <!--<hardwareInterface>EffortJointInterface</hardwareInterface>-->
         <hardwareInterface>PositionJointInterface</hardwareInterface> <!-- TODO: PositionJointInterface? EffortJointInterface?  VelocityJointInterface? -->
       </joint>
-      <actuator name="${prefix}torso_elevation_motor">
+      <actuator name="${prefix}torso_guidance_elevation_motor">
         <mechanicalReduction>1</mechanicalReduction>
         <hardwareInterface>EffortJointInterface</hardwareInterface>
       </actuator>
     </transmission>
-    <link name="${prefix}torso_guidance_slide_link">
+    <link name="${prefix}torso_guidance_elevation_link">
       <visual>
         <origin xyz="0 0 0" rpy="0 0 0"/>
@@ -120,5 +120,5 @@
     <joint name="${prefix}torso_tkd668_joint" type="fixed">
       <origin xyz="0.164 0 0.449" rpy="0 0 0"/>
-      <parent link="${prefix}torso_guidance_slide_link"/>
+      <parent link="${prefix}torso_guidance_elevation_link"/>
       <child link="${prefix}torso_tkd668_link"/>
       <axis xyz="0 0 1"/>

File: vulcano_torso_description/urdf/pantilt/pantilt.urdf.xacro (robot description, xacro)
@@ -3,6 +3,4 @@
   <xacro:property name="PI" value="3.1415926535897931"/>
   <xacro:property name="deg2rad" value="0.01745329251"/>
-  <xacro:property name="elevation_max_longitude" value="0.7"/>
-  <xacro:property name="z_elevation_joint" value="0.442"/>
   <!-- Define the torso -->
   <xacro:macro name="pantilt" params="prefix parent hq">

File: vulcano_torso_description/urdf/vulcano_torso.urdf.xacro (robot description, xacro)
@@ -21,5 +21,5 @@
         <joint name="${prefix}torso_guidance_pantilt_joint" type="fixed">
           <origin xyz="-0.191 0.0 1.178" rpy="0 0 ${180*deg2rad}"/>
-          <parent link="${prefix}torso_guidance_main_link"/>
+          <parent link="${prefix}torso_guidance_revolution_link"/>
           <child link="${prefix}torso_guidance_pantilt_link"/>
           <axis xyz="0 0 1"/>

Commit message: vulcano_torso_description: updated simulation parameters

File: vulcano_torso_description/urdf/guidance/guidance.urdf.xacro (robot description, xacro)
@@ -78,5 +78,4 @@
     </link>
     <joint name="${prefix}torso_guidance_elevation_joint" type="prismatic">
-      <!-- TODO: especificar limites de articulacion y parametros de simulacion -->
       <origin xyz="0 0 0.115" rpy="0 0 0"/>
       <parent link="${prefix}torso_guidance_revolution_link"/>
@@ -84,4 +83,5 @@
       <axis xyz="0 0 1"/>
       <limit lower="0" upper="0.739" effort="100" velocity="100"/>
+      <dynamics friction="1000" damping="1000"/>
     </joint>
 	<transmission name="${prefix}torso_guidance_elevation_trans">

Commit message: vulcano_torso: updated urdf and control file

File: vulcano_torso_description/urdf/guidance/guidance.urdf.xacro (robot description, xacro)
@@ -79,5 +79,5 @@
       <child link="${prefix}torso_guidance_elevation_link"/>
       <axis xyz="0 0 1"/>
-      <limit lower="0" upper="0.739" effort="100" velocity="100"/>
+      <limit lower="0.0" upper="0.68" effort="100" velocity="100"/>
       <dynamics friction="1000" damping="1000"/>
     </joint>

Commit message: vulcano_torso: updated torso controllers and pad

File: vulcano_torso_description/urdf/guidance/guidance.urdf.xacro (robot description, xacro)
@@ -80,5 +80,5 @@
       <axis xyz="0 0 1"/>
       <limit lower="0.0" upper="0.68" effort="100" velocity="100"/>
-      <dynamics friction="1000" damping="1000"/>
+      <dynamics friction="100000" damping="10000"/>
     </joint>
 	<transmission name="${prefix}torso_guidance_elevation_trans">

Commit message: Change torso rotation limits.

File: vulcano_torso_description/urdf/guidance/guidance.urdf.xacro (robot description, xacro)
@@ -40,5 +40,5 @@
       <child link="${prefix}torso_guidance_revolution_link"/>
       <axis xyz="0 0 1"/>
-      <limit lower="${-180*deg2rad}" upper="${180*deg2rad}" effort="100" velocity="0.4"/>
+      <limit lower="${-140*deg2rad}" upper="${220*deg2rad}" effort="100" velocity="0.4"/>
       <dynamics friction="1000" damping="1000"/>
     </joint>

Commit message: Modified torso xacro - Initial real test

File: vulcano_torso_description/urdf/guidance/guidance.urdf.xacro (robot description, xacro)
@@ -114,6 +114,6 @@
     </link>
     <joint name="${prefix}torso_tkd668_joint" type="fixed">
-      <!--origin xyz="0.164 0 0.5015" rpy="0 0 0"/-->
-      <origin xyz="0.164 0 0.449" rpy="0 0 0"/>
+      <origin xyz="0.164 0 0.5015" rpy="0 0 0"/>
+      <!--origin xyz="0.164 0 0.449" rpy="0 0 0"/-->
       <parent link="${prefix}torso_guidance_elevation_link"/>
       <child link="${prefix}torso_tkd668_link"/>

Commit message: Commit local working copy changes.

File: vulcano_torso_description/urdf/guidance/guidance.urdf.xacro (robot description, xacro)
@@ -114,5 +114,6 @@
     </link>
     <joint name="${prefix}torso_tkd668_joint" type="fixed">
-      <origin xyz="0.164 0 0.449" rpy="0 0 0"/>
+      <!--origin xyz="0.164 0 0.449" rpy="0 0 0"/-->
+      <origin xyz="0.164 0 0.5015" rpy="0 0 0"/>
       <parent link="${prefix}torso_guidance_elevation_link"/>
       <child link="${prefix}torso_tkd668_link"/>

Commit message: torso_description: updated model

File: vulcano_torso_description/urdf/guidance/guidance.urdf.xacro (robot description, xacro)
@@ -3,6 +3,9 @@
   <xacro:property name="PI" value="3.1415926535897931"/>
   <xacro:property name="deg2rad" value="0.01745329251"/>
-  <xacro:property name="elevation_max_longitude" value="0.7"/>
-  <xacro:property name="z_elevation_joint" value="0.442"/>
+  <xacro:macro name="cylinder_inertia" params="m r h">
+    <inertia  ixx="${m*(3*r*r+h*h)/12}" ixy = "0" ixz = "0"
+              iyy="${m*(3*r*r+h*h)/12}" iyz = "0"
+              izz="${m*r*r/2}" />
+  </xacro:macro>
   <!-- Define the torso -->
   <xacro:macro name="guidance" params="prefix parent hq">
@@ -13,5 +16,11 @@
       <axis xyz="0 0 1"/>
     </joint>
-    <link name="${prefix}torso_guidance_base_link"/>
+    <link name="${prefix}torso_guidance_base_link">
+      <inertial>
+        <mass value="128" />
+        <origin xyz="0 0 0" />
+        <cylinder_inertia  m="128" r="0.4" h="1.5" /> <!-- TODO: check inertia -->
+      </inertial>
+    </link>
     <joint name="${prefix}torso_guidance_revolution_joint" type="revolute">
       <origin xyz="0 0 0" rpy="0 0 ${PI}"/>
@@ -48,7 +57,7 @@
       </collision>
       <inertial>
-        <origin xyz="0.011 -0.001 0.623" rpy="0 0 0"/>
-        <mass value="128"/>
-        <inertia ixx="29.075" ixy="0.013" ixz="0.582" iyy="28.51" iyz="0.009" izz="1.37"/>
+        <mass value="128" />
+        <origin xyz="0 0 0" />
+        <cylinder_inertia  m="128" r="0.4" h="1.5" /> <!-- TODO: check inertia -->
       </inertial>
     </link>
