Commit message: torso_description: backported new description from kinetic

File: vulcano_torso_description/urdf/guidance/guidance.urdf.xacro (robot description, xacro)
@@ -3,6 +3,9 @@
   <xacro:property name="PI" value="3.1415926535897931"/>
   <xacro:property name="deg2rad" value="0.01745329251"/>
-  <xacro:property name="elevation_max_longitude" value="0.7"/>
-  <xacro:property name="z_elevation_joint" value="0.442"/>
+  <xacro:macro name="cylinder_inertia" params="m r h">
+    <inertia  ixx="${m*(3*r*r+h*h)/12}" ixy = "0" ixz = "0"
+              iyy="${m*(3*r*r+h*h)/12}" iyz = "0"
+              izz="${m*r*r/2}" />
+  </xacro:macro>
   <!-- Define the torso -->
   <xacro:macro name="guidance" params="prefix parent hq">
@@ -14,23 +17,8 @@
     </joint>
     <link name="${prefix}torso_guidance_base_link">
-      <visual>
-        <origin xyz="0 0 0" rpy="0 0 0"/>
-        <geometry>
-          <mesh filename="package://vulcano_torso_description/meshes/guidance/base.stl"/>
-        </geometry>
-       <material name="darkgrey">
-         <color rgba="0.1 0.1 0.1 1"/>
-       </material>
-      </visual>
-      <collision>
-        <origin xyz="0 0 0" rpy="0 0 0"/>
-        <geometry>
-          <mesh filename="package://vulcano_torso_description/meshes/guidance/base.stl"/>
-        </geometry>
-      </collision>
       <inertial>
-        <origin xyz="0 0 -0.152" rpy="0 0 0"/>
-        <mass value="31"/>
-        <inertia ixx="0.404" ixy="0.0" ixz="0.006" iyy="0.403" iyz="0.0" izz="0.34"/>
+        <mass value="128" />
+        <origin xyz="0 0 0" />
+        <cylinder_inertia  m="128" r="0.4" h="1.5" /> <!-- TODO: check inertia -->
       </inertial>
     </link>
@@ -56,5 +44,5 @@
         <origin xyz="0 0 0" rpy="0 0 0"/>
         <geometry>
-          <mesh filename="package://vulcano_torso_description/meshes/guidance/main.stl"/>
+          <mesh filename="package://vulcano_torso_description/meshes/guidance/guidance.stl"/>
         </geometry>
        <material name="darkgrey">
@@ -65,19 +53,19 @@
         <origin xyz="0 0 0" rpy="0 0 0"/>
         <geometry>
-          <mesh filename="package://vulcano_torso_description/meshes/guidance/main.stl"/>
+          <mesh filename="package://vulcano_torso_description/meshes/guidance/guidance.stl"/>
         </geometry>
       </collision>
       <inertial>
-        <origin xyz="0.011 -0.001 0.623" rpy="0 0 0"/>
-        <mass value="128"/>
-        <inertia ixx="29.075" ixy="0.013" ixz="0.582" iyy="28.51" iyz="0.009" izz="1.37"/>
+        <mass value="128" />
+        <origin xyz="0 0 0" />
+        <cylinder_inertia  m="128" r="0.4" h="1.5" /> <!-- TODO: check inertia -->
       </inertial>
     </link>
     <joint name="${prefix}torso_guidance_elevation_joint" type="prismatic">
-      <origin xyz="0 0 0.115" rpy="0 0 0"/>
+      <origin xyz="-0.1687 0 0.720" rpy="0 0 0"/>
       <parent link="${prefix}torso_guidance_revolution_link"/>
       <child link="${prefix}torso_guidance_elevation_link"/>
       <axis xyz="0 0 1"/>
-      <limit lower="0.0" upper="0.68" effort="100" velocity="0.08"/>
+      <limit lower="0.0" upper="0.6" effort="100" velocity="0.08"/>
       <dynamics friction="100000" damping="10000"/>
     </joint>
@@ -113,27 +101,4 @@
       </inertial>
     </link>
-    <joint name="${prefix}torso_tkd668_joint" type="fixed">
-      <origin xyz="0.164 0 0.449" rpy="0 0 0"/>
-      <parent link="${prefix}torso_guidance_elevation_link"/>
-      <child link="${prefix}torso_tkd668_link"/>
-      <axis xyz="0 0 1"/>
-    </joint>
-    <link name="${prefix}torso_tkd668_link">
-      <visual>
-        <origin xyz="0 0 0" rpy="0 0 0"/>
-        <geometry>
-          <mesh filename="package://vulcano_torso_description/meshes/guidance/tkd668.stl"/>
-        </geometry>
-       <material name="darkgrey">
-         <color rgba="0.1 0.1 0.1 1"/>
-       </material>
-      </visual>
-      <collision>
-        <origin xyz="0 0 0" rpy="0 0 0"/>
-        <geometry>
-          <mesh filename="package://vulcano_torso_description/meshes/guidance/tkd668.stl"/>
-        </geometry>
-      </collision>
-    </link>
   </xacro:macro>
 </robot>

File: vulcano_torso_description/urdf/pantilt/pantilt.urdf.xacro (robot description, xacro)
@@ -2,5 +2,4 @@
 <robot xmlns:xacro="http://ros.org/wiki/xacro">
   <xacro:property name="PI" value="3.1415926535897931"/>
-  <xacro:property name="deg2rad" value="0.01745329251"/>
   <!-- Define the torso -->
   <xacro:macro name="pantilt" params="prefix parent hq">
@@ -69,5 +68,5 @@
       <child link="${prefix}torso_pantilt_pan_link"/>
       <axis xyz="0 0 1"/>
-      <limit lower="${-55*deg2rad}" upper="${55*deg2rad}" effort="100" velocity="100"/>
+      <limit lower="-0.95" upper="0.95" effort="100" velocity="100"/>
       <dynamics friction="1000" damping="1000"/>
     </joint>
@@ -106,9 +105,9 @@
     <!-- TILT JOINT/LINK -->
     <joint name="${prefix}torso_pantilt_tilt_joint" type="revolute">
-      <origin xyz="0.0 -0.027 0.0" rpy="${-90*deg2rad} 0 0"/>
+      <origin xyz="0.0 -0.027 0.0" rpy="-1.57 0 0"/>
       <parent link="${prefix}torso_pantilt_pan_link"/>
       <child link="${prefix}torso_pantilt_tilt_base_link"/>
       <axis xyz="0 0 1"/>
-      <limit lower="${-40*deg2rad}" upper="${70*deg2rad}" effort="100" velocity="100"/>
+      <limit lower="-1.26" upper="1.26" effort="100" velocity="100"/>
       <dynamics friction="1000" damping="1000"/>
     </joint>
@@ -147,5 +146,5 @@
     </link>
     <joint name="${prefix}torso_pantilt_tilt_support_joint" type="fixed">
-      <origin xyz="0.0 0.0 0.0" rpy="${90*deg2rad} 0 0"/>
+      <origin xyz="0.0 0.0 0.0" rpy="1.57 0 0"/>
       <parent link="${prefix}torso_pantilt_tilt_base_link"/>
       <child link="${prefix}torso_pantilt_tilt_support_link"/>
@@ -176,5 +175,5 @@
     <joint name="${prefix}torso_pantilt_tilt_fixed_joint" type="fixed">
       <!--<origin xyz="0.0 0.027 0.027" rpy="0 0 0"/>-->
-      <origin xyz="0.0 -0.027 0.027" rpy="${90*deg2rad} 0 0"/>
+      <origin xyz="0.0 -0.027 0.027" rpy="1.57 0 0"/>
       <parent link="${prefix}torso_pantilt_tilt_base_link"/>
       <child link="${prefix}torso_pantilt_tilt_link"/>

Commit message: torso_description: ported from indigo-devel

File: vulcano_torso_description/urdf/guidance/guidance.urdf.xacro (robot description, xacro)
@@ -3,9 +3,6 @@
   <xacro:property name="PI" value="3.1415926535897931"/>
   <xacro:property name="deg2rad" value="0.01745329251"/>
-  <xacro:macro name="cylinder_inertia" params="m r h">
-    <inertia  ixx="${m*(3*r*r+h*h)/12}" ixy = "0" ixz = "0"
-              iyy="${m*(3*r*r+h*h)/12}" iyz = "0"
-              izz="${m*r*r/2}" />
-  </xacro:macro>
+  <xacro:property name="elevation_max_longitude" value="0.7"/>
+  <xacro:property name="z_elevation_joint" value="0.442"/>
   <!-- Define the torso -->
   <xacro:macro name="guidance" params="prefix parent hq">
@@ -17,8 +14,23 @@
     </joint>
     <link name="${prefix}torso_guidance_base_link">
+      <visual>
+        <origin xyz="0 0 0" rpy="0 0 0"/>
+        <geometry>
+          <mesh filename="package://vulcano_torso_description/meshes/guidance/base.stl"/>
+        </geometry>
+       <material name="darkgrey">
+         <color rgba="0.1 0.1 0.1 1"/>
+       </material>
+      </visual>
+      <collision>
+        <origin xyz="0 0 0" rpy="0 0 0"/>
+        <geometry>
+          <mesh filename="package://vulcano_torso_description/meshes/guidance/base.stl"/>
+        </geometry>
+      </collision>
       <inertial>
-        <mass value="128" />
-        <origin xyz="0 0 0" />
-        <cylinder_inertia  m="128" r="0.4" h="1.5" /> <!-- TODO: check inertia -->
+        <origin xyz="0 0 -0.152" rpy="0 0 0"/>
+        <mass value="31"/>
+        <inertia ixx="0.404" ixy="0.0" ixz="0.006" iyy="0.403" iyz="0.0" izz="0.34"/>
       </inertial>
     </link>
@@ -44,5 +56,5 @@
         <origin xyz="0 0 0" rpy="0 0 0"/>
         <geometry>
-          <mesh filename="package://vulcano_torso_description/meshes/guidance/guidance.stl"/>
+          <mesh filename="package://vulcano_torso_description/meshes/guidance/main.stl"/>
         </geometry>
        <material name="darkgrey">
@@ -53,19 +65,19 @@
         <origin xyz="0 0 0" rpy="0 0 0"/>
         <geometry>
-          <mesh filename="package://vulcano_torso_description/meshes/guidance/guidance.stl"/>
+          <mesh filename="package://vulcano_torso_description/meshes/guidance/main.stl"/>
         </geometry>
       </collision>
       <inertial>
-        <mass value="128" />
-        <origin xyz="0 0 0" />
-        <cylinder_inertia  m="128" r="0.4" h="1.5" /> <!-- TODO: check inertia -->
+        <origin xyz="0.011 -0.001 0.623" rpy="0 0 0"/>
+        <mass value="128"/>
+        <inertia ixx="29.075" ixy="0.013" ixz="0.582" iyy="28.51" iyz="0.009" izz="1.37"/>
       </inertial>
     </link>
     <joint name="${prefix}torso_guidance_elevation_joint" type="prismatic">
-      <origin xyz="-0.1687 0 0.720" rpy="0 0 0"/>
+      <origin xyz="0 0 0.115" rpy="0 0 0"/>
       <parent link="${prefix}torso_guidance_revolution_link"/>
       <child link="${prefix}torso_guidance_elevation_link"/>
       <axis xyz="0 0 1"/>
-      <limit lower="0.0" upper="0.6" effort="100" velocity="0.08"/>
+      <limit lower="0.0" upper="0.68" effort="100" velocity="0.08"/>
       <dynamics friction="100000" damping="10000"/>
     </joint>
@@ -101,4 +113,27 @@
       </inertial>
     </link>
+    <joint name="${prefix}torso_tkd668_joint" type="fixed">
+      <origin xyz="0.164 0 0.449" rpy="0 0 0"/>
+      <parent link="${prefix}torso_guidance_elevation_link"/>
+      <child link="${prefix}torso_tkd668_link"/>
+      <axis xyz="0 0 1"/>
+    </joint>
+    <link name="${prefix}torso_tkd668_link">
+      <visual>
+        <origin xyz="0 0 0" rpy="0 0 0"/>
+        <geometry>
+          <mesh filename="package://vulcano_torso_description/meshes/guidance/tkd668.stl"/>
+        </geometry>
+       <material name="darkgrey">
+         <color rgba="0.1 0.1 0.1 1"/>
+       </material>
+      </visual>
+      <collision>
+        <origin xyz="0 0 0" rpy="0 0 0"/>
+        <geometry>
+          <mesh filename="package://vulcano_torso_description/meshes/guidance/tkd668.stl"/>
+        </geometry>
+      </collision>
+    </link>
   </xacro:macro>
 </robot>

File: vulcano_torso_description/urdf/pantilt/pantilt.urdf.xacro (robot description, xacro)
@@ -2,4 +2,5 @@
 <robot xmlns:xacro="http://ros.org/wiki/xacro">
   <xacro:property name="PI" value="3.1415926535897931"/>
+  <xacro:property name="deg2rad" value="0.01745329251"/>
   <!-- Define the torso -->
   <xacro:macro name="pantilt" params="prefix parent hq">
@@ -68,5 +69,5 @@
       <child link="${prefix}torso_pantilt_pan_link"/>
       <axis xyz="0 0 1"/>
-      <limit lower="-0.95" upper="0.95" effort="100" velocity="100"/>
+      <limit lower="${-55*deg2rad}" upper="${55*deg2rad}" effort="100" velocity="100"/>
       <dynamics friction="1000" damping="1000"/>
     </joint>
@@ -105,9 +106,9 @@
     <!-- TILT JOINT/LINK -->
     <joint name="${prefix}torso_pantilt_tilt_joint" type="revolute">
-      <origin xyz="0.0 -0.027 0.0" rpy="-1.57 0 0"/>
+      <origin xyz="0.0 -0.027 0.0" rpy="${-90*deg2rad} 0 0"/>
       <parent link="${prefix}torso_pantilt_pan_link"/>
       <child link="${prefix}torso_pantilt_tilt_base_link"/>
       <axis xyz="0 0 1"/>
-      <limit lower="-1.26" upper="1.26" effort="100" velocity="100"/>
+      <limit lower="${-40*deg2rad}" upper="${70*deg2rad}" effort="100" velocity="100"/>
       <dynamics friction="1000" damping="1000"/>
     </joint>
@@ -146,5 +147,5 @@
     </link>
     <joint name="${prefix}torso_pantilt_tilt_support_joint" type="fixed">
-      <origin xyz="0.0 0.0 0.0" rpy="1.57 0 0"/>
+      <origin xyz="0.0 0.0 0.0" rpy="${90*deg2rad} 0 0"/>
       <parent link="${prefix}torso_pantilt_tilt_base_link"/>
       <child link="${prefix}torso_pantilt_tilt_support_link"/>
@@ -175,5 +176,5 @@
     <joint name="${prefix}torso_pantilt_tilt_fixed_joint" type="fixed">
       <!--<origin xyz="0.0 0.027 0.027" rpy="0 0 0"/>-->
-      <origin xyz="0.0 -0.027 0.027" rpy="1.57 0 0"/>
+      <origin xyz="0.0 -0.027 0.027" rpy="${90*deg2rad} 0 0"/>
       <parent link="${prefix}torso_pantilt_tilt_base_link"/>
       <child link="${prefix}torso_pantilt_tilt_link"/>

File: vulcano_torso_description/urdf/tube_support/tube_support.urdf.xacro (robot description, xacro)
@@ -4,5 +4,5 @@
   <xacro:macro name="tube_support" params="prefix parent *origin *box">
     <joint name="${prefix}tube_support_joint" type="fixed">
-        <xacro:insert_block name="origin" />
+        <insert_block name="origin" />
         <parent link="${parent}" />
         <child link="${prefix}tube_support_link"/>
@@ -12,5 +12,5 @@
         <origin xyz="0 0 0" rpy="0 0 0" />
         <geometry>
-            <xacro:insert_block name="box" />
+            <insert_block name="box" />
         </geometry>
       </collision>

File: vulcano_torso_description/urdf/vulcano_torso.urdf.xacro (robot description, xacro)
@@ -35,11 +35,11 @@
         <xacro:pantilt prefix="${prefix}" parent="${prefix}torso_guidance_pantilt_link" hq="${hq}"/>
         <!-- TODO: check kinect2 position -->
-        <xacro:sensor_kinectv2 prefix="${prefix}torso_kinect" parent="${prefix}torso_pantilt_link" base="true">
+        <xacro:sensor_kinectv2 name="${prefix}torso_kinect" parent="${prefix}torso_pantilt_link" base="true">
             <origin xyz="0.01255 0 0.066" rpy="0 0 0"/>
         </xacro:sensor_kinectv2>
-        <xacro:sensor_ueye_cp_gige prefix="${prefix}torso_ueye_left" parent="${prefix}torso_pantilt_link">
+        <xacro:sensor_ueye_cp_gige name="${prefix}torso_ueye_left" parent="${prefix}torso_pantilt_link">
             <origin xyz="0.0258 -0.14975 0.0165" rpy="0 0 0"/>
         </xacro:sensor_ueye_cp_gige>
-        <xacro:sensor_ueye_cp_gige prefix="${prefix}torso_ueye_right" parent="${prefix}torso_pantilt_link">
+        <xacro:sensor_ueye_cp_gige name="${prefix}torso_ueye_right" parent="${prefix}torso_pantilt_link">
             <origin xyz="0.0258 0.14975 0.0165" rpy="0 0 0"/>
         </xacro:sensor_ueye_cp_gige>
