Commit message: base_description: updated wheel models

File: vulcano_base_description/urdf/vulcano_base.urdf.xacro (robot description, xacro)
@@ -15,8 +15,9 @@
     <!-- Global parameters -->
     <!-- ***************** -->
+    <xacro:property name="vulcano_base_version" value="2.0" />    <!-- x,y,z in translation from base_link to the center of the wheel -->
     <xacro:property name="PI" value="3.1415926535897931"/>
     <xacro:property name="deg2rad" value="0.01745329251"/>
     <!-- Wheel parameters -->
-    <xacro:property name="wheel_offset_x" value="0.467" />    <!-- x,y,z in translation from base_link to the center of the wheel -->
+    <xacro:property name="wheel_offset_x" value="0.6165" />    <!-- x,y,z in translation from base_link to the center of the wheel -->
     <xacro:property name="wheel_offset_y" value="0.285" />
     <xacro:property name="wheel_offset_z" value="0.0" />

File: vulcano_base_description/urdf/wheels/motor_wheel.urdf.xacro (robot description, xacro)
@@ -11,10 +11,10 @@
   <xacro:property name="steer_joint_velocity_limit" value="2" />
   <xacro:property name="steer_joint_position_limit" value="2.9" />
-  <xacro:property name="motor_wheel_mechanical_reduction" value="1.0" />
-  <xacro:property name="wheel_joint_damping" value="0.001" />
-  <xacro:property name="wheel_joint_friction" value="0.001" />
-  <xacro:property name="wheel_joint_effort_limit" value="1000.0" />
-  <xacro:property name="wheel_joint_velocity_limit" value="2000.0" />
-  <xacro:property name="wheel_mechanical_reduction" value="1.0" />
+  <xacro:property name="steer_mechanical_reduction" value="1.0" />
+  <xacro:property name="traction_joint_damping" value="0.001" />
+  <xacro:property name="traction_joint_friction" value="0.001" />
+  <xacro:property name="traction_joint_effort_limit" value="1000.0" />
+  <xacro:property name="traction_joint_velocity_limit" value="6.28" />
+  <xacro:property name="traction_mechanical_reduction" value="1.0" />
   <xacro:macro name="cylinder_inertia" params="m r h">
     <inertia  ixx="${m*(3*r*r+h*h)/12}" ixy = "0" ixz = "0"
@@ -25,7 +25,7 @@
   <!-- TODO: check reflect parameter -->
   <!--MOTOR WHEEL -->
-    <joint name="${prefix}motor_wheel_joint" type="revolute">
+    <joint name="${prefix}wheel_steer_joint" type="revolute">
       <parent link="${parent}"/>
-      <child link="${prefix}motor_wheel"/>
+      <child link="${prefix}wheel_steer_link"/>
       <insert_block name="origin" />
       <axis xyz="0 0 1" rpy="0 0 0" />
@@ -33,15 +33,15 @@
       <joint_properties damping="${steer_joint_damping}" friction="${steer_joint_friction}"/>
     </joint>
-  <transmission name="${prefix}motor_wheel_trans">
+  <transmission name="${prefix}wheel_steer_trans">
      <type>transmission_interface/SimpleTransmission</type>
-     <joint name="${prefix}motor_wheel_joint">
+     <joint name="${prefix}wheel_steer_joint">
         <hardwareInterface>PositionJointInterface</hardwareInterface>
      </joint>
-     <actuator name="${prefix}motor_wheel_motor">
+     <actuator name="${prefix}wheel_steer_motor">
         <hardwareInterface>PositionActuatorInterface</hardwareInterface>
-        <mechanicalReduction>${motor_wheel_mechanical_reduction}</mechanicalReduction>
+        <mechanicalReduction>${steer_mechanical_reduction}</mechanicalReduction>
      </actuator>
   </transmission>
-  <link name="${prefix}motor_wheel">
+  <link name="${prefix}wheel_steer_link">
       <visual>
         <!-- HIGH RESOLUTION WHEELS -->
@@ -88,23 +88,23 @@
     </link>
    <!--WHEEL TIRE -->
-   <joint name="${prefix}wheel_joint" type="continuous">
-        <parent link="${prefix}motor_wheel"/>
-        <child link="${prefix}wheel"/>
+   <joint name="${prefix}wheel_traction_joint" type="continuous">
+        <parent link="${prefix}wheel_steer_link"/>
+        <child link="${prefix}wheel_traction_link"/>
         <origin xyz="0 0 0" rpy="0 0 ${M_PI}" />
         <axis xyz="0 1 0" rpy="0 0 0" />
-        <limit effort="${wheel_joint_effort_limit}" velocity="${wheel_joint_velocity_limit}"/>
-        <joint_properties damping="${wheel_joint_damping}" friction="{wheel_joint_friction}"/>
+        <limit effort="${traction_joint_effort_limit}" velocity="${traction_joint_velocity_limit}"/>
+        <joint_properties damping="${traction_joint_damping}" friction="{traction_joint_friction}"/>
     </joint>
-    <transmission name="${prefix}wheel_trans">
+    <transmission name="${prefix}wheel_traction">
      <type>transmission_interface/SimpleTransmission</type>
-     <joint name="${prefix}wheel_joint">
+     <joint name="${prefix}wheel_traction_joint">
         <hardwareInterface>VelocityJointInterface</hardwareInterface>
      </joint>
-     <actuator name="${prefix}wheel_motor">
+     <actuator name="${prefix}wheel_traction_motor">
        <hardwareInterface>VelocityActuatorInterface</hardwareInterface>
-       <mechanicalReduction>${wheel_mechanical_reduction}</mechanicalReduction>
+       <mechanicalReduction>${traction_mechanical_reduction}</mechanicalReduction>
      </actuator>
     </transmission>
-  <link name="${prefix}wheel">
+  <link name="${prefix}wheel_traction_link">
       <visual>
         <!-- HIGH RESOLUTION WHEELS -->
@@ -147,5 +147,5 @@
       </inertial>
    </link>
-   <!-- gazebo reference="${prefix}wheel">
+   <!-- gazebo reference="${prefix}motor_wheel_link">
         <mu1 value="1.0"/>
         <mu2 value="1.0"/>

Commit message: base_description: updated laser positions

File: vulcano_base_description/urdf/vulcano_base.urdf.xacro (robot description, xacro)
@@ -46,15 +46,9 @@
         </xacro:sensor_imu>
         <xacro:sensor_sick_s300 prefix="${prefix}front_left_laser" parent="${prefix}base_link">
-            <origin xyz="0.606321 0.345821 0.3095" rpy="${180*deg2rad} 0 ${45*deg2rad}"/>
+            <origin xyz="0.75631 0.34581 0.19376" rpy="${180*deg2rad} 0 ${45*deg2rad}"/>
         </xacro:sensor_sick_s300>
         <xacro:sensor_sick_s300 prefix="${prefix}back_right_laser" parent="${prefix}base_link">
-            <origin xyz="-0.606321 -0.345821 0.3095" rpy="${180*deg2rad} 0 ${225*deg2rad}"/>
+            <origin xyz="-0.75631 -0.34581 0.19376" rpy="${180*deg2rad} 0 ${225*deg2rad}"/>
         </xacro:sensor_sick_s300>
-        <joint name="merged_base_laser_joint" type="fixed"> <!-- front and back laser will be merged into this link -->
-            <origin xyz="0 0 0.234" rpy="0 0 0" />
-            <parent link="${prefix}base_link"/>
-            <child link="${prefix}merged_base_laser_link" />
-        </joint>
-        <link name="merged_base_laser_link" />
    </xacro:macro>
 </robot>

Commit message: base_description: corrected laser position

File: vulcano_base_description/urdf/vulcano_base.urdf.xacro (robot description, xacro)
@@ -46,8 +46,8 @@
         </xacro:sensor_imu>
         <xacro:sensor_sick_s300 prefix="${prefix}front_left_laser" parent="${prefix}base_link">
-            <origin xyz="0.75631 0.34581 0.19376" rpy="${180*deg2rad} 0 ${45*deg2rad}"/>
+            <origin xyz="0.75631 0.34581 0.29376" rpy="${180*deg2rad} 0 ${45*deg2rad}"/>
         </xacro:sensor_sick_s300>
         <xacro:sensor_sick_s300 prefix="${prefix}back_right_laser" parent="${prefix}base_link">
-            <origin xyz="-0.75631 -0.34581 0.19376" rpy="${180*deg2rad} 0 ${225*deg2rad}"/>
+            <origin xyz="-0.75631 -0.34581 0.29376" rpy="${180*deg2rad} 0 ${225*deg2rad}"/>
         </xacro:sensor_sick_s300>
    </xacro:macro>

Commit message: base_description: corrected laser positions

File: vulcano_base_description/urdf/vulcano_base.urdf.xacro (robot description, xacro)
@@ -46,8 +46,8 @@
         </xacro:sensor_imu>
         <xacro:sensor_sick_s300 prefix="${prefix}front_left_laser" parent="${prefix}base_link">
-            <origin xyz="0.75631 0.34581 0.29376" rpy="${180*deg2rad} 0 ${45*deg2rad}"/>
+            <origin xyz="0.75631 0.34581 0.30676" rpy="${180*deg2rad} 0 ${45*deg2rad}"/>
         </xacro:sensor_sick_s300>
         <xacro:sensor_sick_s300 prefix="${prefix}back_right_laser" parent="${prefix}base_link">
-            <origin xyz="-0.75631 -0.34581 0.29376" rpy="${180*deg2rad} 0 ${225*deg2rad}"/>
+            <origin xyz="-0.75631 -0.34581 0.30676" rpy="${180*deg2rad} 0 ${225*deg2rad}"/>
         </xacro:sensor_sick_s300>
    </xacro:macro>

Commit message: configuration in progress

File: vulcano_base_description/urdf/vulcano_base.urdf.xacro (robot description, xacro)
@@ -46,8 +46,10 @@
         </xacro:sensor_imu>
         <xacro:sensor_sick_s300 prefix="${prefix}front_left_laser" parent="${prefix}base_link">
-            <origin xyz="0.75631 0.34581 0.30676" rpy="${180*deg2rad} 0 ${45*deg2rad}"/>
+            <!-- origin xyz="0.75631 0.34581 0.30676" rpy="${180*deg2rad} 0 ${135*deg2rad}"/-->
+            <origin xyz="0.826 0.415 0.200" rpy="${180*deg2rad} 0 ${135*deg2rad}"/>
         </xacro:sensor_sick_s300>
         <xacro:sensor_sick_s300 prefix="${prefix}back_right_laser" parent="${prefix}base_link">
-            <origin xyz="-0.75631 -0.34581 0.30676" rpy="${180*deg2rad} 0 ${225*deg2rad}"/>
+            <!-- origin xyz="-0.75631 -0.34581 0.30676" rpy="${180*deg2rad} 0 ${315*deg2rad}"/ -->
+            <origin xyz="-0.826 -0.415 0.200" rpy="${180*deg2rad} 0 ${315*deg2rad}"/>
         </xacro:sensor_sick_s300>
    </xacro:macro>

File: vulcano_torso_description/urdf/guidance/guidance.urdf.xacro (robot description, xacro)
@@ -37,4 +37,5 @@
       </joint>
       <actuator name="${prefix}torso_guidance_revolution_motor">
+        <hardwareInterface>PositionJointInterface</hardwareInterface>
         <mechanicalReduction>1</mechanicalReduction>
       </actuator>
@@ -76,4 +77,5 @@
       </joint>
       <actuator name="${prefix}torso_guidance_elevation_motor">
+        <hardwareInterface>PositionJointInterface</hardwareInterface>
         <mechanicalReduction>1</mechanicalReduction>
       </actuator>

File: vulcano_torso_description/urdf/vulcano_torso.urdf.xacro (robot description, xacro)
@@ -10,5 +10,4 @@
     <xacro:include filename="$(find vulcano_torso_description)/urdf/pantilt/pantilt.urdf.xacro"/>
     <xacro:include filename="$(find vulcano_torso_description)/urdf/tube_support/tube_support.urdf.xacro"/>
-    <xacro:include filename="$(find robotnik_sensors)/urdf/all_sensors.urdf.xacro" />
     <xacro:macro name="vulcano_torso" params="prefix hq"> <!-- TODO: check hq variable -->
         <link name="${prefix}torso_base_link">
@@ -34,14 +33,14 @@
         </link>
         <xacro:pantilt prefix="${prefix}" parent="${prefix}torso_guidance_pantilt_link" hq="${hq}"/>
-        <!-- TODO: check kinect2 position -->
-        <xacro:sensor_kinectv2 prefix="${prefix}torso_kinect" parent="${prefix}torso_pantilt_link" base="true">
+        <!-- TODO: check realsense position -->
+        <xacro:sensor_r430 prefix="${prefix}torso_realsense" parent="${prefix}torso_pantilt_link">
             <origin xyz="0.01255 0 0.066" rpy="0 0 0"/>
-        </xacro:sensor_kinectv2>
-        <xacro:sensor_ueye_cp_gige prefix="${prefix}torso_ueye_left" parent="${prefix}torso_pantilt_link">
+        </xacro:sensor_r430>
+        <!--xacro:sensor_ueye_cp_gige prefix="${prefix}torso_ueye_left" parent="${prefix}torso_pantilt_link">
             <origin xyz="0.0258 -0.14975 0.0165" rpy="0 0 0"/>
         </xacro:sensor_ueye_cp_gige>
         <xacro:sensor_ueye_cp_gige prefix="${prefix}torso_ueye_right" parent="${prefix}torso_pantilt_link">
             <origin xyz="0.0258 0.14975 0.0165" rpy="0 0 0"/>
-        </xacro:sensor_ueye_cp_gige>
+        </xacro:sensor_ueye_cp_gige-->
     </xacro:macro>
 </robot>
